File: Medallion_Board/Medallion_Board.kicad_pcb (KiCad board)
At the start: 2 copper layers, 89 parts, among them IC1 114993121, J1 EXPANSION, J2 RECE.20369.001E.01, P1 JST_ONOFF, P2 JST_PH, P3 JST_BTN_1, P4 JST_BTN_3, P5 JST_BTN_2, Q1 DMG3415U, SW1 KMR2, SW2 KMR2, U1 MDBT50Q-1MV2, U2 MAX17048G_T10, U3 LC86LICMD, U4 RT9080-33GJ5, U5 MCP73831T-2ACI_OT, U6 BNO085, X1 USB4085-GF-A, Y1 32.768KHZ

Commit message: Start PCB design again - compact requirements
Parts:
- removed C29: 100nF, Capacitor_SMD:C_0603_1608Metric
- removed C30, C31: NC, Capacitor_SMD:C_0603_1608Metric
- removed L2: 0R, LQM18DN100M70L:INDC1608X95N
- removed P4: JST_BTN_3, S2B-PH-SM4-TB_LF__SN_:JST_S2B-PH-SM4-TB_LF__SN_
- removed P5: JST_BTN_2, S2B-PH-SM4-TB_LF__SN_:JST_S2B-PH-SM4-TB_LF__SN_
- removed R22: 27R, Resistor_SMD:R_0603_1608Metric
- removed R23: 5.6K, Resistor_SMD:R_0603_1608Metric
- removed R24, R25: 22R, Resistor_SMD:R_0603_1608Metric
- removed SW1, SW2: KMR2, Button_Switch_SMD:SW_Push_1P1T-SH_NO_CK_KMR2xxG
- added BATT1: JST_PH, S2B-PH-SM4-TB_LF__SN_:JST_S2B-PH-SM4-TB_LF__SN_, F.Cu at (156.0, 101.8)
- added ONOFF1: JST_ONOFF, S2B-PH-SM4-TB_LF__SN_:JST_S2B-PH-SM4-TB_LF__SN_, F.Cu at (159.9, 93.2)
- added RESET1: KMR2, Button_Switch_SMD:SW_Push_1P1T-SH_NO_CK_KMR2xxG, F.Cu at (82.5, 32.5)
- C10: value 0.1µF -> 0.1uF
- C11, C13, C9: value 10µF -> 10uF
- C15, C16, C17, C18, C19, C20, C21, C22, C23: value 0.1µF -> 0.1uF; footprint Capacitor_SMD:C_0603_1608Metric -> Capacitor_SMD:C_0402_1005Metric
- C24, C25, C27: value 100nF -> 0.1uF; footprint Capacitor_SMD:C_0603_1608Metric -> Capacitor_SMD:C_0402_1005Metric
- C26: value 22µF -> 22uF; footprint Capacitor_SMD:C_0805_2012Metric -> Capacitor_SMD:C_0402_1005Metric
- C28: value 4.7uF -> 0.1uF; footprint Capacitor_SMD:C_0603_1608Metric -> Capacitor_SMD:C_0402_1005Metric
- CHG1: footprint LED_SMD:LED_0805_2012Metric -> LED_SMD:LED_0603_1608Metric
- IC1: value 114993121 -> Wio-SX1262; footprint Wio-E5-LE:114993121 -> 114993390:114993390
- J1: value EXPANSION -> SWD HEADER; footprint Connector_PinHeader_2.54mm:PinHeader_1x08_P2.54mm_Vertical -> Connector_PinHeader_2.54mm:PinHeader_1x05_P2.54mm_Vertical
- J2: value RECE.20369.001E.01 -> EXPANSION; footprint RECE.20369:RECE20369001E01 -> Connector_PinHeader_2.54mm:PinHeader_1x08_P2.54mm_Vertical
- P1: value JST_ONOFF -> JST_BTN_1
- P2: value JST_PH -> JST_BTN_2
- P3: value JST_BTN_1 -> JST_BTN_3
- R1, R14, R18, R6: value 5.1K -> 5K
- R15: value 0.5K -> 500R
- R17: value 470R -> 5K
- R19: value 5.1K -> 27R
- R20: value 27R -> 10K
- R21: value 10K -> 27R
- R7: value 5.6K -> 5K
- moved U3 197.7 mm to (43.8, 162.2)
- moved R11 195.4 mm to (56.3, 164.2)
- moved R10 192.0 mm to (57.8, 167.2), turned to -90 degrees
- moved R7 189.4 mm to (56.3, 167.2)
- moved U6 177.8 mm to (140.5, 42.0), turned to 90 degrees
- moved R5 166.1 mm to (57.8, 164.2), turned to -90 degrees
- moved C8 164.4 mm to (60.2, 155.7), turned to 180 degrees
- moved C23 161.1 mm to (100.0, 102.0)
- moved D11 160.5 mm to (100.0, 100.0)
- moved J2 160.1 mm to (103.0, 29.4)
- moved D7 159.4 mm to (67.5, 100.0), turned to -90 degrees
- moved C19 158.1 mm to (69.5, 100.0), turned to 90 degrees
- moved D8 155.5 mm to (77.1, 123.0), turned to -45 degrees
- moved C20 154.3 mm to (78.5, 121.5), turned to -45 degrees
- moved D6 148.5 mm to (77.0, 77.0), turned to -135 degrees
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Connections:
- C28 pad 1: 3.3V -> Net-(U6-CAP)
- IC1 pad 1: 3.3V -> /LORA_RF_SW
- IC1 pad 10: Net-(IC1-PB6) -> GND
- IC1 pad 11: unconnected-(IC1-PB5-Pad11) -> /LORA_BUSY
- IC1 pad 12: unconnected-(IC1-PC1-Pad12) -> /LORA_DIO1
- IC1 pad 2: GND -> /SPI_MISO
- IC1 pad 3: unconnected-(IC1-PA13-Pad3) -> /SPI_MOSI
- IC1 pad 4: unconnected-(IC1-PA14-Pad4) -> /SPI_SCK
- IC1 pad 5: unconnected-(IC1-PB15-Pad5) -> /LORA_NRST
- IC1 pad 6: unconnected-(IC1-PA15-Pad6) -> /LORA_NSS
- IC1 pad 7: unconnected-(IC1-PB4-Pad7) -> GND
- IC1 pad 8: unconnected-(IC1-PB3-Pad8) -> 3.3V
- IC1 pad 9: Net-(IC1-PB7) -> unconnected-(IC1-ANT-Pad9)
- J1 pad 1: /GPIO19 -> 3.3V
- J1 pad 2: /GPIO20 -> Net-(J1-SWDCLK)
- J1 pad 3: /GPIO21 -> Net-(J1-SWDIO)
- J1 pad 4: /GPIO22 -> /uC_RESET
- J1 pad 5: /SDA -> GND
- J2 pad 1: GND -> /GPIO14
- J2 pad 2: GND -> /GPIO15
- J2 pad 3: GND -> /GPIO16
- J2 pad 4: GND -> /GPIO17
- P1 pad 1: Net-(U4-EN) -> /USER_BTN_1
- P2 pad 1: VBAT -> /USER_BTN_2
- P3 pad 1: /USER_BTN_1 -> /USER_BTN_3
- R17 pad 1: Net-(R17-Pad1) -> GND
- R17 pad 2: GND -> Net-(X1-CC1)
- R18 pad 2: Net-(X1-CC1) -> Net-(X1-CC2)
- R19 pad 1: GND -> /D+
- R19 pad 2: Net-(X1-CC2) -> Net-(X1-DP1)
- R20 pad 1: /D+ -> Net-(U6-~{BOOT})
- R20 pad 2: Net-(X1-DP1) -> 3.3V
- R21 pad 1: Net-(U6-~{BOOT}) -> /D-
- R21 pad 2: 3.3V -> Net-(X1-DP2)
- U1 pad 10: unconnected-(U1-P0.29/AIN5-Pad10) -> /LORA_DIO1
- U1 pad 12: unconnected-(U1-P0.31/AIN7-Pad12) -> /LORA_RF_SW
- U1 pad 13: unconnected-(U1-P0.28/AIN4-Pad13) -> /LORA_NRST
- U1 pad 14: unconnected-(U1-P0.30/AIN6-Pad14) -> /LORA_BUSY
- U1 pad 36: /RXD_LORA -> /GPIO14
- U1 pad 37: /TXD_LORA -> unconnected-(U1-P0.13-Pad37)
- U1 pad 38: unconnected-(U1-P0.16-Pad38) -> /GPIO16
- U1 pad 39: unconnected-(U1-P0.15-Pad39) -> /GPIO15
- U1 pad 41: unconnected-(U1-P0.17-Pad41) -> /GPIO17
- U1 pad 42: /GPIO19 -> /SPI_SCK
- U1 pad 43: /GPIO21 -> /SPI_MOSI
- U1 pad 44: /GPIO20 -> /LORA_NSS
- U1 pad 46: /GPIO22 -> /SPI_MISO
- U1 pad 51: unconnected-(U1-SWDIO-Pad51) -> Net-(J1-SWDIO)
- U1 pad 53: unconnected-(U1-SWDCLK-Pad53) -> Net-(J1-SWDCLK)
- U1 pad 56: /LORA_RST -> unconnected-(U1-P1.04-Pad56)
- X1 pad S1: Net-(X1-SHELL-PadS1) -> GND
- X1 pad S2: Net-(X1-SHELL-PadS1) -> GND
- X1 pad S3: Net-(X1-SHELL-PadS1) -> GND
- X1 pad S4: Net-(X1-SHELL-PadS1) -> GND
Routing:
- net Net-(X1-DP1): track 0.00 -> 9.85 mm
- net Net-(X1-CC1): track 0.00 -> 9.57 mm, vias 0 -> 1
- net Net-(X1-DP2): track 0.00 -> 8.90 mm, vias 0 -> 1
- net Net-(X1-CC2): track 0.00 -> 5.64 mm
Other:
- board outline added: 70 x 115.3 mm
- copper layers 2 -> 4
