File: Medallion_Board/Medallion_Board.kicad_pcb (KiCad board)
At the start: 4 copper layers, 70 x 70 mm, 84 parts, among them IC1 Wio-SX1262, J1 SWD HEADER, J2 EXPANSION, J3 IPEX, P1 JST_BTN_1, P2 JST_BTN_2, P3 JST_BTN_3, Q1 DMG3415U, U1 MDBT50Q-1MV2, U2 MAX17048G_T10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

Commit message: Move to hierarchical schematic
Parts:
- removed BATT1: JST_PH, S2B-PH-SM4-TB_LF__SN_:JST_S2B-PH-SM4-TB_LF__SN_
- removed C1, C2: 12pF, Capacitor_SMD:C_0402_1005Metric
- removed C10, C15, C16, C17, C18, C19, C20, C21, C22, C23, C24, C25, C27, C28, C7: 0.1uF, Capacitor_SMD:C_0402_1005Metric
- removed C11, C12, C13, C14, C3, C4, C5, C9: 10uF, Capacitor_SMD:C_0805_2012Metric
- removed C26: 22uF, Capacitor_SMD:C_0402_1005Metric
- removed C29, C30: NM, Capacitor_SMD:C_0402_1005Metric
- removed C6: 1uF, Capacitor_SMD:C_0603_1608Metric
- removed C8: 100mF, KW-5R5C104-R:CAPPRD500W60D1000H3150
- removed CHG1: ORANGE, LED_SMD:LED_0603_1608Metric
- removed D1: MBR0540, Diode_SMD:D_SOD-123
- removed D10, D11, D3, D4, D5, D6, D7, D8, D9: WS2812B2020, WS2812B2020:LED_WS2812B2020
- removed D12: TPD1E05U06DPYR, TPD1E05U06DPYR:DIO_TPD1E05U06DPYR
- removed D2: BAV199, BAV199:SOT23
- removed IC1: Wio-SX1262, 114993390:114993390
- removed J1: SWD HEADER, Connector_PinHeader_2.54mm:PinHeader_1x05_P2.54mm_Vertical
- removed J2: EXPANSION, Connector_PinHeader_2.54mm:PinHeader_1x08_P2.54mm_Vertical
- removed J3: IPEX, RECE.20369:RECE20369001E01
- removed L1: 10uH, LQM18DN100M70L:INDC1608X95N
- removed ONOFF1: JST_ONOFF, SM02B-GHS-TB:JST_SM02B-GHS-TB
- removed P1: JST_BTN_1, SM02B-GHS-TB:JST_SM02B-GHS-TB
- removed P2: JST_BTN_2, SM02B-GHS-TB:JST_SM02B-GHS-TB
- removed P3: JST_BTN_3, SM02B-GHS-TB:JST_SM02B-GHS-TB
- removed Q1: DMG3415U, DMG3415U-7:SOT95P240X105-3N
- removed R1, R17, R18, R6, R7: 5K, Resistor_SMD:R_0603_1608Metric
- removed R10, R11, R5: 1K, Resistor_SMD:R_0603_1608Metric
- removed R12, R13, R16, R2, R20, R3: 10K, Resistor_SMD:R_0603_1608Metric
- removed R14: 0R, Resistor_SMD:R_0402_1005Metric
- removed R15: 500R, Resistor_SMD:R_0603_1608Metric
- removed R19, R21: 27R, Resistor_SMD:R_0603_1608Metric
- removed R4, R9: 100K, Resistor_SMD:R_0603_1608Metric
- removed R8: 2K, Resistor_SMD:R_0603_1608Metric
- removed RESET1: KMR2, Button_Switch_SMD:SW_Push_1P1T-SH_NO_CK_KMR2xxG
- removed U1: MDBT50Q-1MV2, MDBT50Q-1MV2:XCVR_MDBT50Q-1MV2
- removed U2: MAX17048G_T10, MAX17048G_T10:SON50P200X200X80-9N
- removed U3: LC86LICMD, LC86LICMD:MODULE_LC86LICMD
- removed U4: RT9080-33GJ5, RT9080-33GJ5:SOT94P280X100-5N
- removed U5: MCP73831T-2ACI_OT, MCP73831T-2ACI_OT:SOT95P280X145-5N
- removed U6: BNO085, BNO085:IC_BNO085
- removed X1: USB4085-GF-A, USB4085-GF-A:GCT_USB4085-GF-A_REVB
- removed Y1: 32.768KHZ, ABS07-32.768KHZ-7-T:XTAL_ABS07-32.768KHZ-7-T
Routing:
- net GND: track 136.9 -> 13.2 mm, vias 41 -> 0
- net /SDA: track 103.7 -> 0.00 mm, vias 6 -> 0
- net /SCL: track 95.9 -> 0.00 mm, vias 6 -> 0
- net Net-(U3-V_BCKP): track 80.1 -> 0.00 mm, vias 4 -> 0
- net /USER_BTN_3: track 74.9 -> 0.00 mm, vias 7 -> 0
- net VBAT: track 312.7 -> 246.0 mm, vias 13 -> 0
- net /NEOPIX: track 66.4 -> 0.00 mm, vias 3 -> 0
- net /LOW_BATT: track 66.2 -> 0.00 mm, vias 2 -> 0
- net /LORA_NRST: track 56.1 -> 0.00 mm, vias 3 -> 0
- net /uC_RESET: track 51.1 -> 0.00 mm, vias 6 -> 0
- net /LORA_BUSY: track 50.6 -> 0.00 mm, vias 5 -> 0
- net /SPI_SCK: track 49.7 -> 0.00 mm, vias 3 -> 0
- net /TXD_GPS: track 47.5 -> 0.00 mm, vias 3 -> 0
- net /LORA_RF_SW: track 47.2 -> 0.00 mm, vias 3 -> 0
- net /LORA_NSS: track 47.1 -> 0.00 mm, vias 3 -> 0
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Other:
- board outline removed
- board text removed: "3.3V"
- board text removed: "GND"
- board text removed: "IO14"
- board text removed: "IO15"
- board text removed: "IO16"
- board text removed: "IO17"
- board text removed: "Jim Wild 2026"
- board text removed: "RST"
- board text removed: "SCL"
- board text removed: "SDA"
- board text removed: "SWDCLK"
- board text removed: "SWDIO"
- board text removed: "v1.0"
