File: Medallion_Board/Medallion_Board.kicad_sch (KiCad schematic)
At the start: 21 parts, among them J1 SWD HEADER, J2 EXPANSION, U1 BMD-340-A-R, U2 MX25R6435FZAIH0, X1 USB4085-GF-A, Y1 32.768KHZ

Commit message: Re-did the layout and routing for the whole board. Added more LEDs, haptics, and properly modelled the e-ink display
Parts:
- U1: AVAILABILITY Unavailable -> (none)
- renumbered R5 to R4, R4 to R5
Connections:
- net GND: now also J1.2 (Pin_2); no longer J1.5 (Pin_5)
- net uC_RESET: now also J1.3 (Pin_3); no longer J1.4 (Pin_4)
- net at U1.43 (SWCLK): now also J1.4 (Pin_4); no longer J1.2 (Pin_2)
- net at U1.44 (SWDIO): now also J1.5 (Pin_5); no longer J1.3 (Pin_3)
- net at R3.2, X1.A6 (DP1): now also X1.B6 (DP2)
- net at R5.2: now also X1.A7 (DN1), X1.B7 (DN2); no longer X1.B6 (DP2)
- net GPS_ANT_ACTIVE: no longer names the net of U1.11 (P0.30)
- net GPS_WAKEUP: no longer names the net of U1.10 (P0.29)
- no-connect marks 15 -> 13
Other:
- sheet Communications ports: added none; removed GPS_ANT_ACTIVE, GPS_WAKEUP
- moved on the sheet: R5
