File: Medallion_Board/user_io.kicad_sch (KiCad schematic)
At the start: 71 parts, among them J3 FH12-24S-0.5SH_55_, P1 JST_BTN_1, P2 JST_BTN_2, P3 JST_BTN_3, Q2 Si1308EDL, U6 BNO085, U7 DRV2605LDGSR

Commit message: Some minor cleaning
Changed lines of the file:
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@@
 		(title "Smart Compass")
 		(date "2026-06-04")
+		(rev "0.2")
 	)
 	(rectangle
@@
 		(property "Value" "GND"
 			(at 161.29 59.69 0)
+			(hide yes)
 			(show_name no)
 			(do_not_autoplace no)
@@
 		(property "Value" "GND"
 			(at 25.4 74.93 0)
+			(hide yes)
 			(show_name no)
 			(do_not_autoplace no)
@@
 		(property "Value" "GND"
 			(at 162.56 44.45 0)
+			(hide yes)
 			(show_name no)
 			(do_not_autoplace no)
@@
 		(property "Value" "GND"
 			(at 64.77 134.62 0)
+			(hide yes)
 			(show_name no)
 			(do_not_autoplace no)
@@
 		(property "Value" "GND"
 			(at 179.07 59.69 0)
+			(hide yes)
 			(show_name no)
 			(do_not_autoplace no)
@@
 		(property "Value" "GND"
 			(at 39.37 148.59 0)
+			(hide yes)
 			(show_name no)
 			(do_not_autoplace no)
@@
 		(property "Value" "GND"
 			(at 97.79 29.21 0)
+			(hide yes)
 			(show_name no)
 			(do_not_autoplace no)
@@
 		(property "Value" "GND"
 			(at 36.83 59.69 0)
+			(hide yes)
 			(show_name no)
 			(do_not_autoplace no)
@@
 		(property "Value" "GND"
 			(at 210.82 113.03 0)
+			(hide yes)
 			(show_name no)
 			(do_not_autoplace no)
@@
 		(property "Value" "GND"
 			(at 125.73 59.69 0)
+			(hide yes)
 			(show_name no)
 			(do_not_autoplace no)
@@
 		(property "Value" "GND"
 			(at 43.18 74.93 0)
+			(hide yes)
 			(show_name no)
 			(do_not_autoplace no)
@@
 		(property "Value" "GND"
 			(at 168.91 29.21 0)
+			(hide yes)
 			(show_name no)
 			(do_not_autoplace no)
@@
 		(property "Value" "GND"
 			(at 19.05 53.34 0)
+			(hide yes)
 			(show_name no)
 			(do_not_autoplace no)
@@
 		(property "Value" "GND"
 			(at 180.34 44.45 0)
+			(hide yes)
 			(show_name no)
 			(do_not_autoplace no)
@@
 		(property "Value" "GND"
 			(at 114.3 74.93 0)
+			(hide yes)
 			(show_name no)
 			(do_not_autoplace no)
@@
 		(property "Value" "GND"
 			(at 151.13 29.21 0)
+			(hide yes)
 			(show_name no)
 			(do_not_autoplace no)
@@
 		(property "Value" "GND"
 			(at 73.66 44.45 0)
+			(hide yes)
 			(show_name no)
 			(do_not_autoplace no)
@@
 		(property "Value" "GND"
 			(at 109.22 44.45 0)
+			(hide yes)
 			(show_name no)
 			(do_not_autoplace no)
@@
 		(property "Value" "GND"
 			(at 91.44 44.45 0)
+			(hide yes)
 			(show_name no)
 			(do_not_autoplace no)
@@
 		(property "Value" "GND"
 			(at 220.98 50.8 0)
+			(hide yes)
 			(show_name no)
 			(do_not_autoplace no)
@@
 		(property "Value" "GND"
 			(at 133.35 29.21 0)
+			(hide yes)
 			(show_name no)
 			(do_not_autoplace no)
@@
 		(property "Value" "GND"
 			(at 19.05 134.62 0)
+			(hide yes)
 			(show_name no)
 			(do_not_autoplace no)
@@
 		(property "Value" "GND"
 			(at 76.2 194.31 0)
+			(hide yes)
 			(show_name no)
 			(do_not_autoplace no)
@@
 		(property "Value" "GND"
 			(at 64.77 115.57 0)
+			(hide yes)
 			(show_name no)
 			(do_not_autoplace no)
@@
 		(property "Value" "GND"
 			(at 107.95 59.69 0)
+			(hide yes)
 			(show_name no)
 			(do_not_autoplace no)
@@
 		(property "Value" "GND"
 			(at 149.86 74.93 0)
+			(hide yes)
 			(show_name no)
 			(do_not_autoplace no)
@@
 		(property "Value" "GND"
 			(at 271.78 49.53 0)
+			(hide yes)
 			(show_name no)
 			(do_not_autoplace no)
@@
 		(property "Value" "GND"
 			(at 167.64 74.93 0)
+			(hide yes)
 			(show_name no)
 			(do_not_autoplace no)
@@
 		(property "Value" "GND"
 			(at 20.32 180.34 0)
+			(hide yes)
 			(show_name no)
 			(do_not_autoplace no)
@@
 		(property "Value" "GND"
 			(at 80.01 29.21 0)
+			(hide yes)
 			(show_name no)
 			(do_not_autoplace no)
@@
 		(property "Value" "GND"
 			(at 127 44.45 0)
+			(hide yes)
 			(show_name no)
 			(do_not_autoplace no)
@@
 		(property "Value" "GND"
 			(at 96.52 74.93 0)
+			(hide yes)
 			(show_name no)
 			(do_not_autoplace no)
@@
 		(property "Value" "GND"
 			(at 54.61 59.69 0)
+			(hide yes)
 			(show_name no)
 			(do_not_autoplace no)
@@
 		(property "Value" "GND"
 			(at 143.51 59.69 0)
+			(hide yes)
 			(show_name no)
 			(do_not_autoplace no)
@@
 		(property "Value" "GND"
 			(at 44.45 29.21 0)
+			(hide yes)
 			(show_name no)
 			(do_not_autoplace no)
@@
 		(property "Value" "GND"
 			(at 77.47 130.81 0)
+			(hide yes)
 			(show_name no)
 			(do_not_autoplace no)
@@
 		(property "Value" "GND"
 			(at 62.23 29.21 0)
+			(hide yes)
 			(show_name no)
 			(do_not_autoplace no)
@@
 		(property "Value" "GND"
 			(at 274.32 124.46 0)
+			(hide yes)
 			(show_name no)
 			(do_not_autoplace no)
@@
 		(property "Value" "GND"
 			(at 60.96 74.93 0)
+			(hide yes)
 			(show_name no)
 			(do_not_autoplace no)
@@
 		(property "Value" "GND"
 			(at 115.57 29.21 0)
+			(hide yes)
 			(show_name no)
 			(do_not_autoplace no)
@@
 		(property "Value" "GND"
 			(at 142.24 140.97 0)
+			(hide yes)
 			(show_name no)
 			(do_not_autoplace no)
@@
 		(property "Value" "GND"
 			(at 55.88 44.45 0)
+			(hide yes)
 			(show_name no)
 			(do_not_autoplace no)
@@
 		(property "Value" "GND"
 			(at 200.66 107.95 0)
+			(hide yes)
 			(show_name no)
 			(do_not_autoplace no)
@@
 		(property "Value" "GND"
 			(at 132.08 74.93 0)
+			(hide yes)
 			(show_name no)
 			(do_not_autoplace no)
@@
 		(property "Value" "GND"
 			(at 78.74 74.93 0)
+			(hide yes)
 			(show_name no)
 			(do_not_autoplace no)
@@
 		(property "Value" "GND"
 			(at 144.78 44.45 0)
+			(hide yes)
 			(show_name no)
 			(do_not_autoplace no)
@@
 		(property "Value" "GND"
 			(at 243.84 55.88 0)
+			(hide yes)
 			(show_name no)
 			(do_not_autoplace no)
@@
 		(property "Value" "GND"
 			(at 90.17 59.69 0)
+			(hide yes)
 			(show_name no)
 			(do_not_autoplace no)
@@
 		(property "Value" "GND"
 			(at 26.67 184.15 0)
+			(hide yes)
 			(show_name no)
 			(do_not_autoplace no)
@@
 		(property "Value" "GND"
 			(at 83.82 194.31 0)
+			(hide yes)
 			(show_name no)
 			(do_not_autoplace no)
@@
 		(property "Value" "GND"
 			(at 72.39 59.69 0)
+			(hide yes)
 			(show_name no)
 			(do_not_autoplace no)

Commit message: review bom and footprints
Parts:
- C24: footprint Capacitor_SMD:C_0402_1005Metric -> Capacitor_SMD:C_0603_1608Metric; MPN GRM158C80E226ME15J -> C0603X5R226M100NTK; PRICE 0.06 -> 0.05187
- C36, C41: MPN C0402X5R475K6R3NTC -> C0402X5R475M100NTC; PRICE 0.0185 -> 0.2223
- Q2: MPN Si1308EDL -> SI1308EDL-EV; PRICE (none) -> 0.32
Changed lines of the file:
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@@
 			)
 		)
-		(property "MPN" "C0402X5R475K6R3NTC"
+		(property "MPN" "C0402X5R475M100NTC"
 			(at 44.45 107.95 90)
 			(hide yes)
@@
 			)
 		)
-		(property "PRICE" "0.0185"
+		(property "PRICE" "0.2223"
 			(at 44.45 107.95 90)
 			(hide yes)
@@
 			)
 		)
-		(property "Datasheet" "https://www.vishay.com/docs/63399/si1308edl.pdf"
+		(property "Datasheet" "https://mm.digikey.com/Volume0/opasdata/d220001/medias/docus/7158/5272_SI1308EDL-EV.pdf"
 			(at 46.99 128.27 0)
 			(hide yes)
@@
 			)
 		)
-		(property "MPN" "Si1308EDL"
+		(property "MPN" "SI1308EDL-EV"
+			(at 41.91 124.46 0)
+			(hide yes)
+			(show_name no)
+			(do_not_autoplace no)
+			(effects
+				(font
+					(size 1.27 1.27)
+				)
+			)
+		)
+		(property "PRICE" "0.32"
 			(at 41.91 124.46 0)
 			(hide yes)
@@
 			)
 		)
-		(property "MPN" "C0402X5R475K6R3NTC"
+		(property "MPN" "C0402X5R475M100NTC"
 			(at 19.05 124.46 90)
 			(hide yes)
@@
 			)
 		)
-		(property "PRICE" "0.0185"
+		(property "PRICE" "0.2223"
 			(at 19.05 124.46 90)
 			(hide yes)
@@
 			)
 		)
-		(property "Footprint" "Capacitor_SMD:C_0402_1005Metric"
+		(property "Footprint" "Capacitor_SMD:C_0603_1608Metric"
 			(at 19.05 44.45 0)
 			(hide yes)
@@
 			)
 		)
-		(property "MPN" "GRM158C80E226ME15J"
+		(property "MPN" "C0603X5R226M100NTK"
 			(at 19.05 44.45 90)
 			(hide yes)
@@
 			)
 		)
-		(property "PRICE" "0.06"
+		(property "PRICE" "0.05187"
 			(at 19.05 44.45 90)
 			(hide yes)

Commit message: Check over i2c, spi, and uart connections
Connections:
- net GND: now also U6.15 (ENV_SCL), U6.16 (ENV_SDA)
- net at U6.17 (SA0/H_MOSI): now also R17.1, U6.18 (~{H_CS}), U6.4 (~{BOOT})
- no-connect marks 8 -> 4
Changed lines of the file:
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@@
 	)
 	(junction
+		(at 262.89 95.25)
+		(diameter 0)
+		(color 0 0 0 0)
+	)
+	(junction
 		(at 232.41 48.26)
 		(diameter 0)
@@
 	)
 	(junction
+		(at 213.36 97.79)
+		(diameter 0)
+		(color 0 0 0 0)
+	)
+	(junction
+		(at 204.47 97.79)
+		(diameter 0)
+		(color 0 0 0 0)
+	)
+	(junction
 		(at 127 22.86)
 		(diameter 0)
@@
 	)
 	(no_connect
-		(at 218.44 107.95)
-	)
-	(no_connect
 		(at 93.98 120.65)
 	)
 	(no_connect
-		(at 218.44 87.63)
-	)
-	(no_connect
 		(at 93.98 118.11)
 	)
 	(no_connect
-		(at 261.62 92.71)
-	)
-	(no_connect
-		(at 261.62 95.25)
-	)
-	(no_connect
 		(at 93.98 137.16)
 	)
@@
 	(wire
 		(pts
+			(xy 218.44 87.63) (xy 204.47 87.63)
+		)
+		(stroke
+			(width 0)
+			(type default)
+		)
+	)
+	(wire
+		(pts
 			(xy 20.32 25.4) (xy 20.32 26.67)
 		)
@@
 	(wire
 		(pts
+			(xy 262.89 92.71) (xy 261.62 92.71)
+		)
+		(stroke
+			(width 0)
+			(type default)
+		)
+	)
+	(wire
+		(pts
 			(xy 133.35 22.86) (xy 133.35 24.13)
 		)
@@
 	(wire
 		(pts
+			(xy 213.36 97.79) (xy 204.47 97.79)
+		)
+		(stroke
+			(width 0)
+			(type default)
+		)
+	)
+	(wire
+		(pts
 			(xy 261.62 82.55) (xy 266.7 82.55)
 		)
@@
 	(wire
 		(pts
+			(xy 261.62 95.25) (xy 262.89 95.25)
+		)
+		(stroke
+			(width 0)
+			(type default)
+		)
+	)
+	(wire
+		(pts
 			(xy 162.56 20.32) (xy 162.56 22.86)
 		)
@@
 	(wire
 		(pts
+			(xy 262.89 96.52) (xy 262.89 95.25)
+		)
+		(stroke
+			(width 0)
+			(type default)
+		)
+	)
+	(wire
+		(pts
 			(xy 73.66 39.37) (xy 73.66 36.83)
 		)
@@
 	(wire
 		(pts
-			(xy 218.44 97.79) (xy 200.66 97.79)
+			(xy 218.44 97.79) (xy 213.36 97.79)
 		)
 		(stroke
@@
 	(wire
 		(pts
+			(xy 213.36 107.95) (xy 213.36 97.79)
+		)
+		(stroke
+			(width 0)
+			(type default)
+		)
+	)
+	(wire
+		(pts
 			(xy 19.05 129.54) (xy 19.05 127)
 		)
@@
 	(wire
 		(pts
+			(xy 204.47 97.79) (xy 200.66 97.79)
+		)
+		(stroke
+			(width 0)
+			(type default)
+		)
+	)
+	(wire
+		(pts
 			(xy 34.29 124.46) (xy 34.29 127)
 		)
@@
 	(wire
 		(pts
+			(xy 204.47 87.63) (xy 204.47 97.79)
+		)
+		(stroke
+			(width 0)
+			(type default)
+		)
+	)
+	(wire
+		(pts
 			(xy 44.45 104.14) (xy 44.45 105.41)
 		)
@@
 	(wire
 		(pts
+			(xy 262.89 95.25) (xy 262.89 92.71)
+		)
+		(stroke
+			(width 0)
+			(type default)
+		)
+	)
+	(wire
+		(pts
 			(xy 17.78 31.75) (xy 16.51 31.75)
 		)
@@
 		)
 	)
+	(wire
+		(pts
+			(xy 218.44 107.95) (xy 213.36 107.95)
+		)
+		(stroke
+			(width 0)
+			(type default)
+		)
+	)
 	(label "PREVGL"
 		(at 73.66 99.06 180)
@@
 					(unit 1)
 				)
+			)
+		)
+	)
+	(symbol
+		(lib_id "power:GND")
+		(at 262.89 96.52 0)
+		(unit 1)
+		(body_style 1)
+		(exclude_from_sim no)
+		(in_bom yes)
+		(on_board yes)
+		(in_pos_files yes)
+		(dnp no)
+		(fields_autoplaced yes)
+		(property "Reference" "#PWR0130"
+			(at 262.89 102.87 0)
+			(hide yes)
+			(show_name no)
+			(do_not_autoplace no)
+			(effects
+				(font
+					(size 1.27 1.27)
+				)
+			)
+		)
+		(property "Value" "GND"
+			(at 262.89 101.6 0)
+			(hide yes)
+			(show_name no)
+			(do_not_autoplace no)
+			(effects
+				(font
+					(size 1.27 1.27)
+				)
+			)
+		)
+		(property "Footprint" ""
+			(at 262.89 96.52 0)
+			(hide yes)
+			(show_name no)
+			(do_not_autoplace no)
+			(effects
+				(font
+					(size 1.27 1.27)
+				)
+			)
+		)
+		(property "Datasheet" ""
+			(at 262.89 96.52 0)
+			(hide yes)
+			(show_name no)
+			(do_not_autoplace no)
+			(effects
+				(font
+					(size 1.27 1.27)
+				)
+			)
+		)
+		(property "Description" "Power symbol creates a global label with name \"GND\" , ground"
+			(at 262.89 96.52 0)
+			(hide yes)
+			(show_name no)
+			(do_not_autoplace no)
+			(effects
+				(font
+					(size 1.27 1.27)
+				)
+			)
+		)
+		(pin "1"
+		)
+		(instances
+			(project "Medallion_Board"
+				(path "/0c161f28-8075-4403-a867-35208f463636/f3daa2fb-5ae8-4cdf-84fa-d6a2260301a1"
+					(reference "#PWR0130")
+					(unit 1)
+				)

Commit message: Re-did the layout and routing for the whole board. Added more LEDs, haptics, and properly modelled the e-ink display
Parts:
- removed C26: 0.1uF, Capacitor_SMD:C_0402_1005Metric, symbol Adafruit ESP32-S3 8MB No PSRAM-eagle-import:CAP_CERAMIC0805-NOOUTLINE
- removed D11: WS2812B2020, WS2812B2020:LED_WS2812B2020, symbol WS2812B2020:WS2812B2020
- J3: value FH12-24S-0.5SH_55_ -> FH12A-24S-0.5SH(55); MPN FH12-24S-0.5SH(55) -> FH12A-24S-0.5SH(55)
- U6: PRICE 13.57 -> 10.06
- renumbered C14 to C15, C15 to C16, C16 to C17, C17 to C18, C18 to C19, C19 to C20, C20 to C21, C21 to C22, C22 to C23, C23 to C24, C24 to C25, C25 to C26, C34 to C27, C33 to C28, C32 to C29, C31 to C30, C30 to C31, C29 to C32, C28 to C33, C27 to C34, D19 to D11, D18 to D12, D17 to D13, D16 to D14, D14 to D16, D13 to D17, D12 to D18, D20 to D19, D21 to D20, D22 to D21
Connections:
- no-connect marks 4 -> 5
Other:
- moved on the sheet: C27, C28, C29, C30, C31, C32, C33, C34, D11, D12, D13, D14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
