File: SmartCompass/SmartCompass.kicad_pcb (KiCad board)
At the start: 4 copper layers, 70 x 70 mm, 124 parts, among them IC1 Wio-SX1262, J1 SWD HEADER, J2 EXPANSION, J3 FH12A-24S-0.5SH(55), J5 IPEX, P1 JST_BTN_1, P2 JST_BTN_2, P3 JST_BTN_3, Q1 DMG3415U, Q2 Si1308EDL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

Commit message: pcb changes
Routing:
- net GND: track 154.2 -> 166.6 mm, vias 87 -> 86
- net /SDA: track 89.5 -> 85.2 mm
- net /SPI_MOSI: track 74.6 -> 76.6 mm
- net /TXD_GPS: track 87.2 -> 88.7 mm
- net /RXD_GPS: track 73.5 -> 74.3 mm
