File: boards/display/Display.kicad_sch (KiCad schematic)
At the start: 20 parts, among them J10 FH12-10S-0.5SH(55), J3 FH12A-24S-0.5SH(55), Q2 Si1308EDL

Commit message: Board migrations. Move to newer LED and IMU
Parts:
- C36, C41: Dielectric (none) -> X5R; DigiKey_PN (none) -> 1276-1482-1-ND; MPN (none) -> CL05A475MP5NRNC; Manufacturer (none) -> Samsung Electro-Mechanics; Voltage (none) -> 10V
- C37, C38, C39, C40, C45: Dielectric (none) -> X7R; DigiKey_PN (none) -> 1276-1184-1-ND; MPN (none) -> CL10B105KA8NNNC; Manufacturer (none) -> Samsung Electro-Mechanics; Voltage (none) -> 25V
- C42: Dielectric (none) -> X7R; DigiKey_PN (none) -> 1276-1184-1-ND; MPN (none) -> CL10B105KA8NNNC; Manufacturer (none) -> Samsung Electro-Mechanics; Sourcing_Note (none) -> Sits on PREVGH at roughly +20V. A 25V X7R has very little m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; Voltage (none) -> 25V
- C43: Dielectric (none) -> X7R; DigiKey_PN (none) -> 1276-1184-1-ND; MPN (none) -> CL10B105KA8NNNC; Manufacturer (none) -> Samsung Electro-Mechanics; Sourcing_Note (none) -> Gate-rail decoupling - check the working voltage against th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; Voltage (none) -> 25V
- C44: Dielectric (none) -> X7R; DigiKey_PN (none) -> 1276-1184-1-ND; MPN (none) -> CL10B105KA8NNNC; Manufacturer (none) -> Samsung Electro-Mechanics; Sourcing_Note (none) -> Sits on PREVGL at roughly -20V. 25V rating is marginal - co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; Voltage (none) -> 25V
- C60: Dielectric (none) -> X5R; DigiKey_PN (none) -> 1276-6456-1-ND; MPN (none) -> CL21A106KPFNNNG; Manufacturer (none) -> Samsung Electro-Mechanics; Voltage (none) -> 10V
- D19, D20, D21: DigiKey_PN (none) -> MBR0540TPMSCT-ND; MPN (none) -> MBR0540-TP; Manufacturer (none) -> MCC (Micro Commercial Components)
- J10: DigiKey_PN (none) -> HFJ110CT-ND; MPN (none) -> FH12-10S-0.5SH(55); Manufacturer (none) -> Hirose Electric Co Ltd
- J3: DigiKey_PN (none) -> HFK124CT-ND; MPN (none) -> FH12A-24S-0.5SH(55); Manufacturer (none) -> Hirose Electric Co Ltd; Sourcing_Note (none) -> Contacts TOP, unlike the FH12-xS parts used for J6/J7/J10 w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
- L1: value 10uH 1A -> 10uH; Current_Rating (none) -> 800mA (750mA Isat); DigiKey_PN (none) -> SRN3015TA-100MCT-ND; MPN (none) -> SRN3015TA-100M; Manufacturer (none) -> Bourns Inc.; Sourcing_Note (none) -> Replaces the NR3015T100M suggested in boards/README.md, whi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
- Q2: DigiKey_PN (none) -> SI1308EDL-T1-GE3CT-ND; MPN (none) -> SI1308EDL-T1-GE3; Manufacturer (none) -> Vishay Siliconix; Sourcing_Note (none) -> Exactly one reel (3000 pcs) in Digi-Key stock and a 55-week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
- R18: DigiKey_PN (none) -> 311-10.0KHRCT-ND; MPN (none) -> RC0603FR-0710KL; Manufacturer (none) -> YAGEO; Tolerance (none) -> 1%
- R19: DigiKey_PN (none) -> 13-RC0603FR-073RLCT-ND; MPN (none) -> RC0603FR-073RL; Manufacturer (none) -> YAGEO; Tolerance (none) -> 1%

Commit message: some more component reworking. Moved to 10 lane ribbon connects between all boards
Parts:
- J3: value FH12A-24S-0.5SH(55) -> FH12-24S-0.5SH(55); DigiKey_PN HFK124CT-ND -> HFJ124CT-ND; MPN FH12A-24S-0.5SH(55) -> FH12-24S-0.5SH(55); Sourcing_Note Contacts TOP, unlike the FH12-xS parts used for J6/J7/J10 w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 -> Contacts BOTTOM, matching J6/J7/J10 so every FFC on the pro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
Other:
- note added: "Decoupling caps and display connector"
- note removed: "Decoupling caps and ribbon cable connector"

Commit message: Update the high voltage caps in the charge pump to higher voltage ones, to give more headroom
Parts:
- C10: renamed from C44; DigiKey_PN 1276-1184-1-ND -> 445-C1608X7R1H105K080ABCT-ND; MPN CL10B105KA8NNNC -> C1608X7R1H105K080AB; Manufacturer Samsung Electro-Mechanics -> TDK; Sourcing_Note Sits on PREVGL at roughly -20V. 25V rating is marginal - co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 -> Sits on PREVGL at roughly -20V. Rated 50V so that DC-bias d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; Tolerance (none) -> 10%; Voltage 25V -> 50V
- C11: renamed from C42; DigiKey_PN 1276-1184-1-ND -> 445-C1608X7R1H105K080ABCT-ND; MPN CL10B105KA8NNNC -> C1608X7R1H105K080AB; Manufacturer Samsung Electro-Mechanics -> TDK; Sourcing_Note Sits on PREVGH at roughly +20V. A 25V X7R has very little m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 -> Sits on PREVGH at roughly +20V. Rated 50V so that DC-bias d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; Tolerance (none) -> 10%; Voltage 25V -> 50V
- renumbered C38 to C1, C60 to C2, C45 to C3, C40 to C4, C37 to C5, C41 to C6, C39 to C7, C43 to C8, C36 to C9, D19 to D1, D20 to D2, D21 to D3, J10 to J1, J3 to J2, Q2 to Q1, R18 to R1, R19 to R2
Other:
- note added: "Interface to main board"
- note removed: "1 +3.3V 2 GND 3 SPI_SCK 4 SPI_MOSI 5 GND"
- note removed: "6 DISP_CS 7 DISP_DC 8 DISP_RES 9 DISP_BUSY 10 GND"
- note removed: "Interface to main board -- J10, 10-pin 0.5mm FFC:"
- note removed: "SCK and MOSI are flanked by GND; the slow signals sit at the far end."
- moved on the sheet: C10, C9, D2

Commit message: Update inductors. However, one still needs a footprint
Parts:
- L1: footprint Inductor_SMD:L_Taiyo-Yuden_NR-30xx -> (none)
Changed lines of the file:
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@@
 			)
 		)
-		(property "Footprint" "Inductor_SMD:L_Taiyo-Yuden_NR-30xx"
+		(property "Footprint" ""
 			(at 128.27 77.47 0)
 			(hide yes)

Commit message: UPGRADE 1UF CAPACITORS
Parts:
- C1, C3, C4, C5, C7: DigiKey_PN 1276-1184-1-ND -> 445-C1608X7R1H105K080ABCT-ND; MPN CL10B105KA8NNNC -> C1608X7R1H105K080AB; Manufacturer Samsung Electro-Mechanics -> TDK; Tolerance (none) -> 10%; Voltage 25V -> 50V
- C8: DigiKey_PN 1276-1184-1-ND -> 445-C1608X7R1H105K080ABCT-ND; MPN CL10B105KA8NNNC -> C1608X7R1H105K080AB; Manufacturer Samsung Electro-Mechanics -> TDK; Sourcing_Note Gate-rail decoupling - check the working voltage against th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 -> Gate-rail decoupling. Rated 50V so DC-bias derating at the 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; Tolerance (none) -> 10%; Voltage 25V -> 50V
Changed lines of the file:
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@@
 			)
 		)
-		(property "Datasheet" ""
+		(property "Datasheet" "https://product.tdk.com/system/files/dam/doc/product/capacitor/ceramic/mlcc/catalog/mlcc_commercial_general_en.pdf"
 			(at 132.08 181.61 0)
 			(hide yes)
@@
 			)
 		)
-		(property "MPN" "CL10B105KA8NNNC"
+		(property "MPN" "C1608X7R1H105K080AB"
 			(at 132.08 181.61 0)
 			(hide yes)
@@
 			)
 		)
-		(property "Manufacturer" "Samsung Electro-Mechanics"
+		(property "Manufacturer" "TDK"
 			(at 132.08 181.61 0)
 			(hide yes)
@@
 			)
 		)
-		(property "DigiKey_PN" "1276-1184-1-ND"
+		(property "DigiKey_PN" "445-C1608X7R1H105K080ABCT-ND"
 			(at 132.08 181.61 0)
 			(hide yes)
@@
 			)
 		)
-		(property "Voltage" "25V"
+		(property "Voltage" "50V"
 			(at 132.08 181.61 0)
 			(hide yes)
@@
 			)
 		)
-		(property "Sourcing_Note" "Gate-rail decoupling - check the working voltage against the SSD1681 reference circuit, 25V is marginal."
+		(property "Sourcing_Note" "Gate-rail decoupling. Rated 50V so DC-bias derating at the gate-rail working voltage still leaves useful capacitance; the 25V part previously fitted here was marginal."
 			(at 132.08 181.61 0)
 			(hide yes)
@@
 			)
 		)
+    (property "Tolerance" "10%" (at 132.08 181.61 0)
+      (effects (font (size 1.27 1.27)) (hide yes))
+    )
 		(pin "1"
 		)
@@
 			)
 		)
-		(property "Datasheet" ""
+		(property "Datasheet" "https://product.tdk.com/system/files/dam/doc/product/capacitor/ceramic/mlcc/catalog/mlcc_commercial_general_en.pdf"
 			(at 95.25 190.5 0)
 			(hide yes)
@@
 			)
 		)
-		(property "MPN" "CL10B105KA8NNNC"
+		(property "MPN" "C1608X7R1H105K080AB"
 			(at 95.25 190.5 0)
 			(hide yes)
@@
 			)
 		)
-		(property "Manufacturer" "Samsung Electro-Mechanics"
+		(property "Manufacturer" "TDK"
 			(at 95.25 190.5 0)
 			(hide yes)
@@
 			)
 		)
-		(property "DigiKey_PN" "1276-1184-1-ND"
+		(property "DigiKey_PN" "445-C1608X7R1H105K080ABCT-ND"
 			(at 95.25 190.5 0)
 			(hide yes)
@@
 			)
 		)
-		(property "Voltage" "25V"
+		(property "Voltage" "50V"
 			(at 95.25 190.5 0)
 			(hide yes)
@@
 			)
 		)
+    (property "Tolerance" "10%" (at 95.25 190.5 0)
+      (effects (font (size 1.27 1.27)) (hide yes))
+    )
 		(pin "1"
 		)
@@
 			)
 		)
-		(property "Datasheet" ""
+		(property "Datasheet" "https://product.tdk.com/system/files/dam/doc/product/capacitor/ceramic/mlcc/catalog/mlcc_commercial_general_en.pdf"
 			(at 132.08 171.45 0)
 			(hide yes)
@@
 			)
 		)
-		(property "MPN" "CL10B105KA8NNNC"
+		(property "MPN" "C1608X7R1H105K080AB"
 			(at 132.08 171.45 0)
 			(hide yes)
@@
 			)
 		)
-		(property "Manufacturer" "Samsung Electro-Mechanics"
+		(property "Manufacturer" "TDK"
 			(at 132.08 171.45 0)
 			(hide yes)
@@
 			)
 		)
-		(property "DigiKey_PN" "1276-1184-1-ND"
+		(property "DigiKey_PN" "445-C1608X7R1H105K080ABCT-ND"
 			(at 132.08 171.45 0)
 			(hide yes)
@@
 			)
 		)
-		(property "Voltage" "25V"
+		(property "Voltage" "50V"
 			(at 132.08 171.45 0)
 			(hide yes)
@@
 			)
 		)
+    (property "Tolerance" "10%" (at 132.08 171.45 0)
+      (effects (font (size 1.27 1.27)) (hide yes))
+    )
 		(pin "1"
 		)
@@
 			)
 		)
-		(property "Datasheet" ""
+		(property "Datasheet" "https://product.tdk.com/system/files/dam/doc/product/capacitor/ceramic/mlcc/catalog/mlcc_commercial_general_en.pdf"
 			(at 107.95 176.53 0)
 			(hide yes)
@@
 			)
 		)
-		(property "MPN" "CL10B105KA8NNNC"
+		(property "MPN" "C1608X7R1H105K080AB"
 			(at 107.95 176.53 0)
 			(hide yes)
@@
 			)
 		)
-		(property "Manufacturer" "Samsung Electro-Mechanics"
+		(property "Manufacturer" "TDK"
 			(at 107.95 176.53 0)
 			(hide yes)
@@
 			)
 		)
-		(property "DigiKey_PN" "1276-1184-1-ND"
+		(property "DigiKey_PN" "445-C1608X7R1H105K080ABCT-ND"
 			(at 107.95 176.53 0)
 			(hide yes)
@@
 			)
 		)
-		(property "Voltage" "25V"
+		(property "Voltage" "50V"
 			(at 107.95 176.53 0)
 			(hide yes)
@@
 			)
 		)
+    (property "Tolerance" "10%" (at 107.95 176.53 0)
+      (effects (font (size 1.27 1.27)) (hide yes))
+    )
 		(pin "1"
 		)
@@
 			)
 		)
-		(property "Datasheet" ""
+		(property "Datasheet" "https://product.tdk.com/system/files/dam/doc/product/capacitor/ceramic/mlcc/catalog/mlcc_commercial_general_en.pdf"
 			(at 114.3 166.37 0)
 			(hide yes)
@@
 			)
 		)
-		(property "MPN" "CL10B105KA8NNNC"
+		(property "MPN" "C1608X7R1H105K080AB"
 			(at 114.3 166.37 0)
 			(hide yes)
@@
 			)
 		)
-		(property "Manufacturer" "Samsung Electro-Mechanics"
+		(property "Manufacturer" "TDK"
 			(at 114.3 166.37 0)
 			(hide yes)
@@
 			)
 		)
-		(property "DigiKey_PN" "1276-1184-1-ND"
+		(property "DigiKey_PN" "445-C1608X7R1H105K080ABCT-ND"
 			(at 114.3 166.37 0)
 			(hide yes)
@@
 			)
 		)
-		(property "Voltage" "25V"
+		(property "Voltage" "50V"
 			(at 114.3 166.37 0)
 			(hide yes)
@@
 			)
 		)
+    (property "Tolerance" "10%" (at 114.3 166.37 0)
+      (effects (font (size 1.27 1.27)) (hide yes))
+    )
 		(pin "1"
 		)
@@
 			)
 		)
-		(property "Datasheet" ""
+		(property "Datasheet" "https://product.tdk.com/system/files/dam/doc/product/capacitor/ceramic/mlcc/catalog/mlcc_commercial_general_en.pdf"
 			(at 58.42 168.91 0)
 			(hide yes)
@@
 			)
 		)
-		(property "MPN" "CL10B105KA8NNNC"
+		(property "MPN" "C1608X7R1H105K080AB"
 			(at 58.42 168.91 0)
 			(hide yes)
@@
 			)
 		)
-		(property "Manufacturer" "Samsung Electro-Mechanics"
+		(property "Manufacturer" "TDK"
 			(at 58.42 168.91 0)
 			(hide yes)
@@
 			)
 		)
-		(property "DigiKey_PN" "1276-1184-1-ND"
+		(property "DigiKey_PN" "445-C1608X7R1H105K080ABCT-ND"
 			(at 58.42 168.91 0)
 			(hide yes)
@@
 			)
 		)
-		(property "Voltage" "25V"
+		(property "Voltage" "50V"
 			(at 58.42 168.91 0)
 			(hide yes)
@@
 			)
 		)
+    (property "Tolerance" "10%" (at 58.42 168.91 0)
+      (effects (font (size 1.27 1.27)) (hide yes))
+    )
 		(pin "1"
 		)

Commit message: Update the MOSFET to something more modern
Parts:
- removed Q1: Si1308EDL, Package_TO_SOT_SMD:SOT-323_SC-70, symbol Transistor_FET:Si1308EDL
- added Q1: IRLML6346, Package_TO_SOT_SMD:SOT-23, symbol Transistor_FET:Q_NMOS_GSD
Connections:
- net EPD_SW: now also Q1.3 (D)
- net GDR: now also Q1.1 (G)
- net RESE: now also Q1.2 (S)
Changed lines of the file:
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@@
-	)
-	(symbol
-		(lib_id "Transistor_FET:Si1308EDL")
-		(at 149.86 87.63 0)
-		(unit 1)
-		(body_style 1)
-		(exclude_from_sim no)
-		(in_bom yes)
-		(on_board yes)
-		(in_pos_files yes)
-		(dnp no)
-		(property "Reference" "Q1"
-			(at 158.496 86.106 0)
-			(show_name no)
-			(do_not_autoplace no)
-			(effects
-				(font
-					(size 1.27 1.27)
-				)
-				(justify left)
-			)
-		)
-		(property "Value" "Si1308EDL"
-			(at 155.448 88.646 0)
-			(show_name no)
-			(do_not_autoplace no)
-			(effects
-				(font
-					(size 1.27 1.27)
-				)
-				(justify left)
-			)
-		)
-		(property "Footprint" "Package_TO_SOT_SMD:SOT-323_SC-70"
-			(at 154.94 85.725 0)
-			(hide yes)
-			(show_name no)
-			(do_not_autoplace no)
-			(effects
-				(font
-					(size 1.27 1.27)
-					(italic yes)
-				)
-				(justify left)
-			)
-		)
-		(property "Datasheet" "https://www.vishay.com/docs/63399/si1308edl.pdf"
-			(at 154.94 83.82 0)
-			(hide yes)
-			(show_name no)
-			(do_not_autoplace no)
-			(effects
-				(font
-					(size 1.27 1.27)
-				)
-				(justify left)
-			)
-		)
-		(property "Description" "30V Vds, 1.4A Id, N-Channel MOSFET, SC-70"
-			(at 149.86 87.63 0)
-			(hide yes)
-			(show_name no)
-			(do_not_autoplace no)
-			(effects
-				(font
-					(size 1.27 1.27)
-				)
-			)
-		)
-		(property "MPN" "SI1308EDL-T1-GE3"
-			(at 149.86 87.63 0)
-			(hide yes)
-			(show_name no)
-			(do_not_autoplace no)
-			(effects
-				(font
-					(size 1.27 1.27)
-				)
-			)
-		)
-		(property "Manufacturer" "Vishay Siliconix"
-			(at 149.86 87.63 0)
-			(hide yes)
-			(show_name no)
-			(do_not_autoplace no)
-			(effects
-				(font
-					(size 1.27 1.27)
-				)
-			)
-		)
-		(property "DigiKey_PN" "SI1308EDL-T1-GE3CT-ND"
-			(at 149.86 87.63 0)
-			(hide yes)
-			(show_name no)
-			(do_not_autoplace no)
-			(effects
-				(font
-					(size 1.27 1.27)
-				)
-			)
-		)
-		(property "Sourcing_Note" "Exactly one reel (3000 pcs) in Digi-Key stock and a 55-week factory lead - the longest on the whole design. Worth identifying a second source for any build beyond prototypes."
-			(at 149.86 87.63 0)
-			(hide yes)
-			(show_name no)
-			(do_not_autoplace no)
-			(effects
-				(font
-					(size 1.27 1.27)
-				)
-			)
-		)
-		(pin "1"
-		)
-		(pin "2"
-		)
-		(pin "3"
-		)
-		(instances
-			(project "Display"
-				(path "/5bea690c-773f-4a31-824a-9096c0b28e28"
-					(reference "Q1")
-					(unit 1)
-				)
-			)
-		)
 	)
 	(symbol
@@
 		)
 	)
-	(sheet_instances
+	  (symbol (lib_id "Transistor_FET:Q_NMOS_GSD") (at 149.86 87.63 0) (unit 1)
+    (body_style 1) (exclude_from_sim no) (in_bom yes) (on_board yes) (in_pos_files yes) (dnp no)
+    (property "Reference" "Q1"
+      (at 154.94 89.535 0)
+      (show_name no)
+      (do_not_autoplace no)
+      (effects
+    				(font
+    					(size 1.27 1.27)
+    				)
+    				(justify left)
+    			)
+    )
+    (property "Value" "IRLML6346"
+      (at 154.94 87.63 0)
+      (show_name no)
+      (do_not_autoplace no)
+      (effects
+    				(font
+    					(size 1.27 1.27)
+    				)
+    				(justify left)
+    			)
+    )
+    (property "Footprint" "Package_TO_SOT_SMD:SOT-23"
+      (at 154.94 90.17 0)
+      (hide yes)
+      (show_name no)
+      (do_not_autoplace no)
+      (effects
+    				(font
+    					(size 1.27 1.27)
+    				)
+    			)
+    )
+    (property "Datasheet" "https://www.infineon.com/assets/row/public/documents/24/49/infineon-irlml6346-datasheet-en.pdf"
+      (at 149.86 87.63 0)
+      (hide yes)
+      (show_name no)
+      (do_not_autoplace no)
+      (effects
+    				(font
+    					(size 1.27 1.27)
+    				)
+    			)
+    )
+    (property "Description" "30V Vds, 3.4A Id, 63mOhm N-Channel logic-level MOSFET, SOT-23"
+      (at 149.86 87.63 0)
+      (hide yes)
+      (show_name no)
+      (do_not_autoplace no)
+      (effects
+    				(font
+    					(size 1.27 1.27)
+    				)
+    			)
+    )
+    (property "MPN" "IRLML6346TRPBF" (at 149.86 87.63 0)
+      (effects (font (size 1.27 1.27)) (hide yes))
+    )
+    (property "Manufacturer" "Infineon Technologies" (at 149.86 87.63 0)
+      (effects (font (size 1.27 1.27)) (hide yes))
+    )
+    (property "DigiKey_PN" "IRLML6346TRPBFCT-ND" (at 149.86 87.63 0)
+      (effects (font (size 1.27 1.27)) (hide yes))
+    )
+    (property "Sourcing_Note" "Replaces the Si1308EDL, which had a 55-week factory lead and a single reel in Digi-Key stock. Chosen for gate drive rather than current: Vgs(th) 1.1 V max with Rds(on) specified down to 2.5 V of gate drive (80 mOhm), so it is fully enhanced from the driver IC's 3.3 V GDR output. Its gate is a heavier load than the Si1308EDL's - Qg 2.9 nC against 1.4 nC typ, Ciss 270 pF against 105 pF, both at 4.5 V - but it matches the Si1304BDL that the panel datasheet's reference circuit offers as its own alternative (Qg 2.7 nC at 4.5 V), so it is within what the GDR output is expected to drive. Peak switch current is set by the 3 ohm sense resistor on RESE and is far below this part's rating, so the current rating is not the binding constraint. ~105,000 in stock, 20-week lead. Qualified second source: Toshiba SSM3K376R, a lighter gate still (Qg 2.2 nC, Ciss 200 pF), but it is SOT-23F flat-lead and would want its own land pattern." (at 149.86 87.63 0)
+      (effects (font (size 1.27 1.27)) (hide yes))
+    )
+    (pin "1")
+    (pin "2")
+    (pin "3")
+    (instances
+      (project "Display"
+        (path "/5bea690c-773f-4a31-824a-9096c0b28e28"
+          (reference "Q1")
+          (unit 1)
+        )
+      )
+    )
+  )
+  (sheet_instances
 		(path "/"
 			(page "1")
