File: boards/main/SmartCompass.kicad_sch (KiCad schematic)
At the start: 21 parts, among them J1 SWD HEADER, J2 EXPANSION, U1 BMD-340-A-R, U2 MX25R6435FZAIH0, X1 USB4085-GF-A, Y1 32.768KHZ

Commit message: Board migrations. Move to newer LED and IMU
Parts:
- C1, C2: Dielectric (none) -> X5R; DigiKey_PN (none) -> 1276-6456-1-ND; Manufacturer (none) -> Samsung Electro-Mechanics; Voltage (none) -> 10V
- C3, C4: Dielectric (none) -> C0G; DigiKey_PN (none) -> 1276-1178-1-ND; MPN C0402C0G120J500NTB -> CL05C120JB5NNNC; Manufacturer (none) -> Samsung Electro-Mechanics; Voltage (none) -> 50V
- C5: Dielectric (none) -> X7R; DigiKey_PN (none) -> 1276-1184-1-ND; MPN 0603B105K100XD -> CL10B105KA8NNNC; Manufacturer (none) -> Samsung Electro-Mechanics; Voltage (none) -> 25V
- C6: Dielectric (none) -> X7R; DigiKey_PN (none) -> 1276-6844-1-ND; MPN 0402B104K160HI -> CL05B104KO5VPNC; Manufacturer (none) -> Samsung Electro-Mechanics; Voltage (none) -> 16V
- R1, R2, R4: value 5K -> 5.1K; DigiKey_PN (none) -> 311-5.10KHRCT-ND; MPN RT0603BRE075KL -> RC0603FR-075K1L; Manufacturer (none) -> YAGEO; Tolerance (none) -> 1%
- R3, R5, R6, R7: Manufacturer (none) -> YAGEO; Tolerance (none) -> 1%
- R8: DigiKey_PN (none) -> 311-10.0KHRCT-ND; Manufacturer (none) -> YAGEO; Tolerance (none) -> 1%
- RESET1: DigiKey_PN (none) -> CKN10244CT-ND; Manufacturer (none) -> C&K
- U1: DigiKey_PN (none) -> 672-BMD-340-A-RCT-ND; Manufacturer (none) -> u-blox
- U2: DigiKey_PN (none) -> 1092-1173-ND; Manufacturer (none) -> Macronix; Sourcing_Note (none) -> Digi-Key stock 0, 52-week factory lead. Every 4x4 USON vari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
- X1: DigiKey_PN (none) -> 2073-USB4085-GF-ACT-ND; Manufacturer (none) -> GCT
- Y1: DigiKey_PN (none) -> 535-9543-1-ND; Manufacturer (none) -> Abracon LLC
Changed lines of the file:
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@@
 			)
 		)
-		(property "Value" "5K"
+		(property "Value" "5.1K"
 			(at 256.54 68.58 0)
 			(show_name no)
@@
 			)
 		)
-		(property "Description" ""
+		(property "Description" "USB-C CC1 pulldown (Rd), 5.1k per USB Type-C spec"
 			(at 256.54 68.58 0)
 			(hide yes)
@@
 			)
 		)
-		(property "MPN" "RT0603BRE075KL"
+		(property "MPN" "RC0603FR-075K1L"
 			(at 256.54 68.58 0)
 			(hide yes)
@@
 			)
 		)
+    (property "Manufacturer" "YAGEO" (at 256.54 68.58 0)
+      (effects (font (size 1.27 1.27)) (hide yes))
+    )
+    (property "DigiKey_PN" "311-5.10KHRCT-ND" (at 256.54 68.58 0)
+      (effects (font (size 1.27 1.27)) (hide yes))
+    )
+    (property "Tolerance" "1%" (at 256.54 68.58 0)
+      (effects (font (size 1.27 1.27)) (hide yes))
+    )
 		(pin "2"
 		)
@@
 			)
 		)
-		(property "MPN" "C0402C0G120J500NTB"
+		(property "MPN" "CL05C120JB5NNNC"
 			(at 48.26 57.15 90)
 			(hide yes)
@@
 			)
 		)
+    (property "Manufacturer" "Samsung Electro-Mechanics" (at 48.26 57.15 0)
+      (effects (font (size 1.27 1.27)) (hide yes))
+    )
+    (property "DigiKey_PN" "1276-1178-1-ND" (at 48.26 57.15 0)
+      (effects (font (size 1.27 1.27)) (hide yes))
+    )
+    (property "Voltage" "50V" (at 48.26 57.15 0)
+      (effects (font (size 1.27 1.27)) (hide yes))
+    )
+    (property "Dielectric" "C0G" (at 48.26 57.15 0)
+      (effects (font (size 1.27 1.27)) (hide yes))
+    )
 		(pin "1"
 		)
@@
 			)
 		)
+    (property "Manufacturer" "Samsung Electro-Mechanics" (at 127.0 26.67 0)
+      (effects (font (size 1.27 1.27)) (hide yes))
+    )
+    (property "DigiKey_PN" "1276-6456-1-ND" (at 127.0 26.67 0)
+      (effects (font (size 1.27 1.27)) (hide yes))
+    )
+    (property "Voltage" "10V" (at 127.0 26.67 0)
+      (effects (font (size 1.27 1.27)) (hide yes))
+    )
+    (property "Dielectric" "X5R" (at 127.0 26.67 0)
+      (effects (font (size 1.27 1.27)) (hide yes))
+    )
 		(pin "1"
 		)
@@
 			)
 		)
+    (property "Manufacturer" "YAGEO" (at 128.27 92.71 0)
+      (effects (font (size 1.27 1.27)) (hide yes))
+    )
+    (property "Tolerance" "1%" (at 128.27 92.71 0)
+      (effects (font (size 1.27 1.27)) (hide yes))
+    )
 		(pin "1"
 		)
@@
 			)
 		)
+    (property "Manufacturer" "C&K" (at 203.2 96.52 0)
+      (effects (font (size 1.27 1.27)) (hide yes))
+    )
+    (property "DigiKey_PN" "CKN10244CT-ND" (at 203.2 96.52 0)
+      (effects (font (size 1.27 1.27)) (hide yes))
+    )
 		(pin "1"
 		)
@@
 			)
 		)
+    (property "Manufacturer" "u-blox" (at 97.79 69.85 0)
+      (effects (font (size 1.27 1.27)) (hide yes))
+    )
+    (property "DigiKey_PN" "672-BMD-340-A-RCT-ND" (at 97.79 69.85 0)
+      (effects (font (size 1.27 1.27)) (hide yes))
+    )
 		(pin "1"
 		)
@@
 			)
 		)
+    (property "Manufacturer" "Samsung Electro-Mechanics" (at 138.43 26.67 0)
+      (effects (font (size 1.27 1.27)) (hide yes))
+    )
+    (property "DigiKey_PN" "1276-6456-1-ND" (at 138.43 26.67 0)
+      (effects (font (size 1.27 1.27)) (hide yes))
+    )
+    (property "Voltage" "10V" (at 138.43 26.67 0)
+      (effects (font (size 1.27 1.27)) (hide yes))
+    )
+    (property "Dielectric" "X5R" (at 138.43 26.67 0)
+      (effects (font (size 1.27 1.27)) (hide yes))
+    )
 		(pin "1"
 		)
@@
 			)
 		)
+    (property "Manufacturer" "YAGEO" (at 254.0 77.47 0)
+      (effects (font (size 1.27 1.27)) (hide yes))
+    )
+    (property "Tolerance" "1%" (at 254.0 77.47 0)
+      (effects (font (size 1.27 1.27)) (hide yes))
+    )
 		(pin "2"
 		)
@@
 			)
 		)
+    (property "Manufacturer" "YAGEO" (at 227.33 129.54 0)
+      (effects (font (size 1.27 1.27)) (hide yes))
+    )
+    (property "DigiKey_PN" "311-10.0KHRCT-ND" (at 227.33 129.54 0)
+      (effects (font (size 1.27 1.27)) (hide yes))
+    )
+    (property "Tolerance" "1%" (at 227.33 129.54 0)
+      (effects (font (size 1.27 1.27)) (hide yes))
+    )
 		(pin "1"
 		)
@@
 			)
 		)
-		(property "Value" "5K"
+		(property "Value" "5.1K"
 			(at 203.2 82.55 0)
 			(show_name no)
@@
 			)
 		)
-		(property "MPN" "RT0603BRE075KL"
+		(property "MPN" "RC0603FR-075K1L"
 			(at 203.2 82.55 0)
 			(hide yes)
@@
 			)
 		)
+    (property "Manufacturer" "YAGEO" (at 203.2 82.55 0)
+      (effects (font (size 1.27 1.27)) (hide yes))
+    )
+    (property "DigiKey_PN" "311-5.10KHRCT-ND" (at 203.2 82.55 0)
+      (effects (font (size 1.27 1.27)) (hide yes))
+    )
+    (property "Tolerance" "1%" (at 203.2 82.55 0)
+      (effects (font (size 1.27 1.27)) (hide yes))
+    )
 		(pin "1"
 		)
@@
 			)
 		)
-		(property "MPN" "0402B104K160HI"
+		(property "MPN" "CL05B104KO5VPNC"
 			(at 267.97 146.05 90)
 			(hide yes)
@@
 			)
 		)
+    (property "Manufacturer" "Samsung Electro-Mechanics" (at 267.97 146.05 0)
+      (effects (font (size 1.27 1.27)) (hide yes))
+    )
+    (property "DigiKey_PN" "1276-6844-1-ND" (at 267.97 146.05 0)
+      (effects (font (size 1.27 1.27)) (hide yes))
+    )
+    (property "Voltage" "16V" (at 267.97 146.05 0)
+      (effects (font (size 1.27 1.27)) (hide yes))
+    )
+    (property "Dielectric" "X7R" (at 267.97 146.05 0)
+      (effects (font (size 1.27 1.27)) (hide yes))
+    )
 		(pin "1"
 		)
@@
 			)
 		)
-		(property "Description" "32.768 kHz ±20ppm Crystal 7pF 70 kOhms 2-SMD, No Lead"
+		(property "Description" "32.768 kHz +/-20ppm, CL=7pF, 3.2x1.5mm"
 			(at 54.61 50.8 0)
 			(hide yes)
@@
 			)
 		)
+    (property "Manufacturer" "Abracon LLC" (at 54.61 50.8 0)
+      (effects (font (size 1.27 1.27)) (hide yes))
+    )
+    (property "DigiKey_PN" "535-9543-1-ND" (at 54.61 50.8 0)
+      (effects (font (size 1.27 1.27)) (hide yes))
+    )
 		(pin "1"
 		)
@@
 			)
 		)
+    (property "Manufacturer" "YAGEO" (at 128.27 95.25 0)
+      (effects (font (size 1.27 1.27)) (hide yes))
+    )
+    (property "Tolerance" "1%" (at 128.27 95.25 0)
+      (effects (font (size 1.27 1.27)) (hide yes))
+    )
 		(pin "1"
 		)
@@
 			)
 		)
-		(property "Value" "5K"
+		(property "Value" "5.1K"
 			(at 256.54 71.12 0)
 			(show_name no)
@@
 			)
 		)
-		(property "Description" ""
+		(property "Description" "USB-C CC2 pulldown (Rd), 5.1k per USB Type-C spec"
 			(at 256.54 71.12 0)
 			(hide yes)
@@
 			)
 		)
-		(property "MPN" "RT0603BRE075KL"
+		(property "MPN" "RC0603FR-075K1L"
 			(at 256.54 71.12 0)
 			(hide yes)
@@
 			)
 		)
+    (property "Manufacturer" "YAGEO" (at 256.54 71.12 0)
+      (effects (font (size 1.27 1.27)) (hide yes))
+    )
+    (property "DigiKey_PN" "311-5.10KHRCT-ND" (at 256.54 71.12 0)
+      (effects (font (size 1.27 1.27)) (hide yes))
+    )
+    (property "Tolerance" "1%" (at 256.54 71.12 0)
+      (effects (font (size 1.27 1.27)) (hide yes))
+    )
 		(pin "1"
 		)
@@
 			)
 		)
-		(property "MPN" "0603B105K100XD"
+		(property "MPN" "CL10B105KA8NNNC"
 			(at 210.82 97.79 90)
 			(hide yes)
@@
 			)
 		)
+    (property "Manufacturer" "Samsung Electro-Mechanics" (at 210.82 97.79 0)
+      (effects (font (size 1.27 1.27)) (hide yes))
+    )
+    (property "DigiKey_PN" "1276-1184-1-ND" (at 210.82 97.79 0)
+      (effects (font (size 1.27 1.27)) (hide yes))
+    )
+    (property "Voltage" "25V" (at 210.82 97.79 0)
+      (effects (font (size 1.27 1.27)) (hide yes))
+    )
+    (property "Dielectric" "X7R" (at 210.82 97.79 0)
+      (effects (font (size 1.27 1.27)) (hide yes))
+    )
 		(pin "1"
 		)
@@
 			)
 		)
-		(property "MPN" "C0402C0G120J500NTB"
+		(property "MPN" "CL05C120JB5NNNC"
 			(at 48.26 44.45 90)
 			(hide yes)
@@
 			)
 		)
+    (property "Manufacturer" "Samsung Electro-Mechanics" (at 48.26 44.45 0)
+      (effects (font (size 1.27 1.27)) (hide yes))
+    )
+    (property "DigiKey_PN" "1276-1178-1-ND" (at 48.26 44.45 0)
+      (effects (font (size 1.27 1.27)) (hide yes))
+    )
+    (property "Voltage" "50V" (at 48.26 44.45 0)
+      (effects (font (size 1.27 1.27)) (hide yes))
+    )
+    (property "Dielectric" "C0G" (at 48.26 44.45 0)
+      (effects (font (size 1.27 1.27)) (hide yes))
+    )
 		(pin "1"
 		)
@@
 			)
 		)
+    (property "Manufacturer" "Macronix" (at 248.92 146.05 0)
+      (effects (font (size 1.27 1.27)) (hide yes))
+    )
+    (property "DigiKey_PN" "1092-1173-ND" (at 248.92 146.05 0)
+      (effects (font (size 1.27 1.27)) (hide yes))
+    )
+    (property "Sourcing_Note" "Digi-Key stock 0, 52-week factory lead. Every 4x4 USON variant is unstocked; the only stocked MX25R6435F is MX25R6435FZNIL0 (1092-1201-ND) in 8-WSON 6x5mm, which needs a different footprint and PCB rework." (at 248.92 146.05 0)
+      (effects (font (size 1.27 1.27)) (hide yes))
+    )
 		(pin "1"
 		)
@@
 			)
 		)
+    (property "Manufacturer" "YAGEO" (at 254.0 82.55 0)
+      (effects (font (size 1.27 1.27)) (hide yes))
+    )
+    (property "Tolerance" "1%" (at 254.0 82.55 0)
+      (effects (font (size 1.27 1.27)) (hide yes))
+    )
 		(pin "2"
 		)
@@
 			)
 		)
+    (property "Manufacturer" "GCT" (at 236.22 82.55 0)
+      (effects (font (size 1.27 1.27)) (hide yes))
+    )
+    (property "DigiKey_PN" "2073-USB4085-GF-ACT-ND" (at 236.22 82.55 0)
+      (effects (font (size 1.27 1.27)) (hide yes))
+    )
 		(pin "A5"
 		)

Commit message: some more component reworking. Moved to 10 lane ribbon connects between all boards
Parts:
- C1, C2, C3, C4, C6: symbol Adafruit ESP32-S3 8MB No PSRAM-eagle-import:CAP_CERAMIC0805-NOOUTLINE -> smart_compass_main:CAP_CERAMIC0805-NOOUTLINE
- C5: symbol Adafruit ESP32-S3 8MB No PSRAM-eagle-import:CAP_CERAMIC0603_NO -> smart_compass_main:CAP_CERAMIC0603_NO
- R1, R2, R3, R4, R5, R6, R7, R8: symbol Adafruit ESP32-S3 8MB No PSRAM-eagle-import:RESISTOR_0603_NOOUT -> smart_compass_main:RESISTOR_0603_NOOUT
- RESET1: symbol Adafruit ESP32-S3 8MB No PSRAM-eagle-import:SWITCH_TACT_SMT4.6X2.8 -> smart_compass_main:SWITCH_TACT_SMT4.6X2.8
- U1: symbol BMD-340-A-R:BMD-340-A-R -> smart_compass_main:BMD-340-A-R
- U2: value MX25R6435FZAIH0 -> S25FL064LABNFI043; footprint MX25R6435FZAIH0:SON80P400X400X60-9N -> smart_compass:SON80P400X400X60-9N; symbol MX25R6435FZAIH0:MX25R6435FZAIH0 -> smart_compass_main:S25FL064L; DigiKey_PN 1092-1173-ND -> 448-S25FL064LABNFI043CT-ND; MANUFACTURER Macronix -> Infineon Technologies; MF Macronix -> Infineon Technologies; MP MX25R6435FZAIH0 -> S25FL064LABNFI043; MPN MX25R6435FZAIH0 -> S25FL064LABNFI043; Manufacturer Macronix -> Infineon Technologies; PRICE 2.04 -> 1.67; Purchase-URL https://www.snapeda.com/api/url_track_click_mouser/?unipart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 -> https://www.digikey.com/en/products/detail/infineon-technol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; Sourcing_Note Digi-Key stock 0, 52-week factory lead. Every 4x4 USON vari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 -> Replaces MX25R6435FZAIH0 (Digi-Key stock 0, 52-week lead; f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
- X1: symbol USB4085-GF-A:USB4085-GF-A -> smart_compass_main:USB4085-GF-A
- Y1: symbol ABS07-32.768KHZ-7-T:ABS07-32.768KHZ-7-T -> smart_compass_main:ABS07-32.768KHZ-7-T
Other:
- note added: "From the datasheet Section 11.5 (Power-up and power-down): Please note that a pull-up resistor on CS# may ensure a safe and proper power-up/down level."
- note removed: "From the datasheet Section 12: Please note that a pull-up resistor on CS# may ensure a safe and proper power-up/down level."

Commit message: Add a voltage booster and logic shift to the LED ring. Power consumption implications, but necessary
Parts:
- U1: footprint BMD_340_A_R:RIGADO_BMD-340-A-R -> (none)
- U2: footprint smart_compass:SON80P400X400X60-9N -> (none)
- X1: footprint USB4085-GF-A:GCT_USB4085-GF-A_REVB -> (none)
- Y1: footprint ABS07-32.768KHZ-7-T:XTAL_ABS07-32.768KHZ-7-T -> (none)
Connections:
- net RING_EN: now reaches U1.56 (P1.00)
- no-connect marks 14 -> 13
Other:
- sheet User IO ports: added RING_EN; removed none
Changed lines of the file:
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@@
 	)
 	(junction
+		(at 203.2 91.44)
+		(diameter 0)
+		(color 0 0 0 0)
+	)
+	(junction
 		(at 118.11 140.97)
 		(diameter 0)
@@
 	)
 	(junction
+		(at 203.2 101.6)
+		(diameter 0)
+		(color 0 0 0 0)
+	)
+	(junction
 		(at 54.61 44.45)
 		(diameter 0)
@@
 	)
 	(no_connect
-		(at 113.03 39.37)
-	)
-	(no_connect
 		(at 113.03 77.47)
 	)
@@
 	(wire
 		(pts
+			(xy 179.07 41.91) (xy 194.31 41.91)
+		)
+		(stroke
+			(width 0)
+			(type default)
+		)
+	)
+	(wire
+		(pts
 			(xy 203.2 88.9) (xy 203.2 91.44)
 		)
@@
 		)
 	)
+	(label "RING_EN"
+		(at 194.31 41.91 0)
+		(effects
+			(font
+				(size 1.27 1.27)
+			)
+			(justify left bottom)
+		)
+	)
 	(label "GPIO19"
 		(at 177.8 135.89 0)
@@
 		)
 	)
+	(label "RING_EN"
+		(at 113.03 39.37 0)
+		(effects
+			(font
+				(size 1.27 1.27)
+			)
+			(justify left bottom)
+		)
+	)
 	(label "SCL"
 		(at 44.45 110.49 0)
@@
 		(dnp no)
 		(fields_autoplaced yes)
-		(property "Reference" "#PWR05"
+		(property "Reference" "#PWR06"
 			(at 138.43 35.56 0)
 			(hide yes)
@@
 			(project "SmartCompass"
 				(path "/0c161f28-8075-4403-a867-35208f463636"
-					(reference "#PWR05")
+					(reference "#PWR06")
 					(unit 1)
 				)
@@
 			)
 		)
-		(property "Footprint" "BMD_340_A_R:RIGADO_BMD-340-A-R"
+		(property "Footprint" ""
 			(at 97.79 69.85 0)
 			(hide yes)
@@
 			)
 		)
-		(property "Footprint" "ABS07-32.768KHZ-7-T:XTAL_ABS07-32.768KHZ-7-T"
+		(property "Footprint" ""
 			(at 54.61 50.8 0)
 			(hide yes)
@@
 		(dnp no)
 		(fields_autoplaced yes)
-		(property "Reference" "#PWR04"
+		(property "Reference" "#PWR05"
 			(at 132.08 35.56 0)
 			(hide yes)
@@
 			(project "SmartCompass"
 				(path "/0c161f28-8075-4403-a867-35208f463636"
-					(reference "#PWR04")
+					(reference "#PWR05")
 					(unit 1)
 				)
@@
 		(dnp no)
 		(fields_autoplaced yes)
-		(property "Reference" "#PWR06"
+		(property "Reference" "#PWR04"
 			(at 78.74 34.29 0)
 			(hide yes)
@@
 			(project "SmartCompass"
 				(path "/0c161f28-8075-4403-a867-35208f463636"
-					(reference "#PWR06")
+					(reference "#PWR04")
 					(unit 1)
 				)
@@
 			)
 		)
-		(property "Footprint" "smart_compass:SON80P400X400X60-9N"
+		(property "Footprint" ""
 			(at 248.92 146.05 0)
 			(hide yes)
@@
 			)
 		)
-		(property "Footprint" "USB4085-GF-A:GCT_USB4085-GF-A_REVB"
+		(property "Footprint" ""
 			(at 236.22 82.55 0)
 			(hide yes)
@@
 			(effects
 				(font
+					(size 1.27 1.27)
+				)
+				(justify left)
+			)
+		)
+		(pin "RING_EN" input
+			(at 179.07 41.91 0)
+			(effects
+				(font

Commit message: Update the footprint for the flash chip
Parts:
- U2: footprint (none) -> Package_DFN_QFN:DFN-8-1EP_4x4mm_P0.8mm_EP2.3x3.24mm
Changed lines of the file:
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@@
 	(text "From the datasheet\nSection 11.5 (Power-up and power-down):\nPlease note that a pull-up resistor\non CS# may ensure a safe and proper \npower-up/down level."
 		(exclude_from_sim no)
-		(at 247.396 123.698 0)
+		(at 256.032 122.936 0)
 		(effects
 			(font
@@
 	)
 	(junction
+		(at 267.97 138.43)
+		(diameter 0)
+		(color 0 0 0 0)
+	)
+	(junction
 		(at 118.11 133.35)
 		(diameter 0)
@@
 	)
 	(junction
-		(at 267.97 138.43)
-		(diameter 0)
-		(color 0 0 0 0)
-	)
-	(junction
 		(at 207.01 104.14)
 		(diameter 0)
@@
 	(wire
 		(pts
-			(xy 267.97 128.27) (xy 267.97 138.43)
+			(xy 267.97 135.89) (xy 267.97 138.43)
 		)
 		(stroke
@@
 	)
 	(label "RING_EN"
-		(at 194.31 41.91 0)
+		(at 194.31 41.91 180)
 		(effects
 			(font
 				(size 1.27 1.27)
 			)
-			(justify left bottom)
+			(justify right bottom)
 		)
 	)
@@
 		)
 		(property "REV" "C"
-			(at 267.97 146.05 0)
+			(at 266.954 146.812 0)
+			(hide yes)
 			(show_name no)
 			(do_not_autoplace no)
@@
 	(symbol
 		(lib_id "power:+3.3V")
-		(at 267.97 128.27 0)
+		(at 267.97 135.89 0)
 		(unit 1)
 		(body_style 1)
@@
 		(fields_autoplaced yes)
 		(property "Reference" "#PWR016"
-			(at 267.97 132.08 0)
+			(at 267.97 139.7 0)
 			(hide yes)
 			(show_name no)
@@
 		)
 		(property "Value" "+3.3V"
-			(at 267.97 123.19 0)
+			(at 267.97 130.81 0)
 			(show_name no)
 			(do_not_autoplace no)
@@
 		)
 		(property "Footprint" ""
-			(at 267.97 128.27 0)
+			(at 267.97 135.89 0)
 			(hide yes)
 			(show_name no)
@@
 		)
 		(property "Datasheet" ""
-			(at 267.97 128.27 0)
+			(at 267.97 135.89 0)
 			(hide yes)
 			(show_name no)
@@
 		)
 		(property "Description" "Power symbol creates a global label with name \"+3.3V\""
-			(at 267.97 128.27 0)
+			(at 267.97 135.89 0)
 			(hide yes)
 			(show_name no)
@@
 			)
 		)
-		(property "Footprint" ""
+		(property "Footprint" "Package_DFN_QFN:DFN-8-1EP_4x4mm_P0.8mm_EP2.3x3.24mm"
 			(at 248.92 146.05 0)
 			(hide yes)
@@
 					(size 1.27 1.27)
 				)
-				(justify left)
+				(justify right)
 			)
 		)

Commit message: UPGRADE 1UF CAPACITORS
Parts:
- C5: DigiKey_PN 1276-1184-1-ND -> 445-C1608X7R1H105K080ABCT-ND; MPN CL10B105KA8NNNC -> C1608X7R1H105K080AB; Manufacturer Samsung Electro-Mechanics -> TDK; PRICE 0.05765 -> 0.0615; Tolerance (none) -> 10%; Voltage 25V -> 50V
Changed lines of the file:
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@@
 			)
 		)
-		(property "Datasheet" ""
+		(property "Datasheet" "https://product.tdk.com/system/files/dam/doc/product/capacitor/ceramic/mlcc/catalog/mlcc_commercial_general_en.pdf"
 			(at 210.82 97.79 0)
 			(hide yes)
@@
 			)
 		)
-		(property "MPN" "CL10B105KA8NNNC"
+		(property "MPN" "C1608X7R1H105K080AB"
 			(at 210.82 97.79 90)
 			(hide yes)
@@
 			)
 		)
-		(property "PRICE" "0.05765"
+		(property "PRICE" "0.0615"
 			(at 210.82 97.79 90)
 			(hide yes)
@@
 			)
 		)
-		(property "Manufacturer" "Samsung Electro-Mechanics"
+		(property "Manufacturer" "TDK"
 			(at 210.82 97.79 0)
 			(hide yes)
@@
 			)
 		)
-		(property "DigiKey_PN" "1276-1184-1-ND"
+		(property "DigiKey_PN" "445-C1608X7R1H105K080ABCT-ND"
 			(at 210.82 97.79 0)
 			(hide yes)
@@
 			)
 		)
-		(property "Voltage" "25V"
+		(property "Voltage" "50V"
 			(at 210.82 97.79 0)
 			(hide yes)
@@
 			)
 		)
+    (property "Tolerance" "10%" (at 210.82 97.79 0)
+      (effects (font (size 1.27 1.27)) (hide yes))
+    )
 		(pin "1"
 		)

Commit message: grab a bunch of datasheets. Fix some models, fix some footprints, replace an unsuited capacitor
Parts:
- U2: MANUFACTURER Infineon Technologies -> (none)
- Y1: MANUFACTURER Abracon -> (none)

Commit message: exclude non-populated symbols from the BOM
Parts:
- J1, J2: now left out of the parts list
Changed lines of the file:
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@@
 		(body_style 1)
 		(exclude_from_sim no)
-		(in_bom yes)
+		(in_bom no)
 		(on_board yes)
 		(in_pos_files yes)
@@
 		(body_style 1)
 		(exclude_from_sim no)
-		(in_bom yes)
+		(in_bom no)
 		(on_board yes)
 		(in_pos_files yes)
