File: boards/main/communications.kicad_sch (KiCad schematic)
At the start: 15 parts, among them IC1 Wio-SX1262, J5 IPEX, U8 MAX-M10S-00B

Commit message: Grab missing footprints and models, and assign them to symbols
Parts:
- AE1: footprint (none) -> smart_compass:ANT_1575AT_JOT
- D2: footprint (none) -> smart_compass:DIO_TPD1E05U06DPYR
- IC1: footprint (none) -> smart_compass:MODULE12P-1.27-11X11.6MM
- J5: footprint (none) -> smart_compass:SMT_9.001E.01_TAL
- U8: footprint (none) -> smart_compass:XCVR_MAX-M10S-00B

Commit message: replace capacitor that's in danger of being a bottleneck
Parts:
- C22, C24: DigiKey_PN 1276-6456-1-ND -> 445-6970-1-ND; MPN CL21A106KPFNNNG -> CGA4J3X5R1A106K125AB; Manufacturer Samsung Electro-Mechanics -> TDK; PRICE 0.07 -> 0.24

Commit message: Fixing symbols
Connections:
- net GND: now also J5.1 (GND_1), J5.2 (GND_2), J5.3 (GND_3)
- net at C25.1, J5.4 (CENTRE), R18.1: now also D2.2 (GND)
Other:
- moved on the sheet: D2, R22

Commit message: Initial placements of main board components. Also set some trace rules
Connections:
- net GPS_EXT: now reaches C25.1, D2.2 (GND), J5.4 (CENTRE), R18.1
- net GPS_RF: now reaches C26.1, R18.2, R22.1, U8.11 (RF_IN)
- net GPS_ANT: now reaches AE1.1 (FEED), R22.2
