File: boards/main/power.kicad_sch (KiCad schematic)
At the start: 19 parts, among them Q1 DMP2045U, U3 RT9080-33GJ5, U4 MCP73831T-2ACI_OT, U5 MAX17048G_T10

Commit message: Fix missing/incorrect digikey numbers
Parts:
- R11: DigiKey_PN (none) -> 311-3.90KHRCT-ND
- R12, R9: DigiKey_PN (none) -> 311-100KHRCT-ND
Changed lines of the file:
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@@
 			)
 		)
+    (property "DigiKey_PN" "311-100KHRCT-ND" (at 153.67 63.5 0)
+      (effects (font (size 1.27 1.27)) (hide yes))
+    )
 		(pin "1"
 		)
@@
 			)
 		)
+    (property "DigiKey_PN" "311-100KHRCT-ND" (at 181.61 39.37 0)
+      (effects (font (size 1.27 1.27)) (hide yes))
+    )
 		(pin "2"
 		)
@@
 			)
 		)
+    (property "DigiKey_PN" "311-3.90KHRCT-ND" (at 44.45 62.23 0)
+      (effects (font (size 1.27 1.27)) (hide yes))
+    )
 		(pin "1"
 		)

Commit message: Use proper flash footprint and model. Also swap out deprecated resistor on the main board
Parts:
- R10: DigiKey_PN 311-5.10KHRCT-ND -> P5.10KHCT-ND; MPN RC0603FR-075K1L -> ERJ-3EKF5101V; Manufacturer YAGEO -> Panasonic
Changed lines of the file:
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@@
 			)
 		)
-    (property "DigiKey_PN" "311-100KHRCT-ND" (at 153.67 63.5 0)
-      (effects (font (size 1.27 1.27)) (hide yes))
-    )
+		(property "DigiKey_PN" "311-100KHRCT-ND"
+			(at 153.67 63.5 0)
+			(hide yes)
+			(show_name no)
+			(do_not_autoplace no)
+			(effects
+				(font
+					(size 1.27 1.27)
+				)
+			)
+		)
 		(pin "1"
 		)
@@
 			)
 		)
-		(property "Manufacturer" "JST"
-			(at 224.79 41.91 0)
-			(hide yes)
-			(show_name no)
-			(do_not_autoplace no)
-			(effects
-				(font
-					(size 1.27 1.27)
-				)
-				(justify bottom)
-			)
-		)
 		(property "MPN" "S2B-PH-SM4-TB"
 			(at 224.79 41.91 0)
@@
 			)
 		)
-    (property "DigiKey_PN" "311-100KHRCT-ND" (at 181.61 39.37 0)
-      (effects (font (size 1.27 1.27)) (hide yes))
-    )
+		(property "DigiKey_PN" "311-100KHRCT-ND"
+			(at 181.61 39.37 0)
+			(hide yes)
+			(show_name no)
+			(do_not_autoplace no)
+			(effects
+				(font
+					(size 1.27 1.27)
+				)
+			)
+		)
 		(pin "2"
 		)
@@
 			)
 		)
-    (property "DigiKey_PN" "311-3.90KHRCT-ND" (at 44.45 62.23 0)
-      (effects (font (size 1.27 1.27)) (hide yes))
-    )
+		(property "DigiKey_PN" "311-3.90KHRCT-ND"
+			(at 44.45 62.23 0)
+			(hide yes)
+			(show_name no)
+			(do_not_autoplace no)
+			(effects
+				(font
+					(size 1.27 1.27)
+				)
+			)
+		)
 		(pin "1"
 		)
@@
 			)
 		)
-		(property "Datasheet" "https://yageogroup.com/content/datasheet/asset/file/PYU-RC_GROUP_51_ROHS_L"
+		(property "Datasheet" "https://industrial.panasonic.com/cdbs/www-data/pdf/RDA0000/AOA0000C304.pdf"
 			(at 78.74 41.91 0)
 			(hide yes)
@@
 			)
 		)
-		(property "MPN" "RC0603FR-075K1L"
+		(property "MPN" "ERJ-3EKF5101V"
 			(at 78.74 41.91 0)
 			(hide yes)
@@
 			)
 		)
-		(property "Manufacturer" "YAGEO"
+		(property "Manufacturer" "Panasonic"
 			(at 78.74 41.91 0)
 			(hide yes)
@@
 			)
 		)
-		(property "DigiKey_PN" "311-5.10KHRCT-ND"
+		(property "DigiKey_PN" "P5.10KHCT-ND"
 			(at 78.74 41.91 0)
 			(hide yes)

Commit message: Grab missing footprints and models, and assign them to symbols
Parts:
- BATT1: footprint (none) -> smart_compass:JST_S2B-PH-SM4-TB
- U3: footprint (none) -> smart_compass:SOT94P280X100-5N
- U4: footprint (none) -> smart_compass:SOT95P280X145-5N
- U5: footprint (none) -> smart_compass:SON50P200X200X80-9N
Changed lines of the file:
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@@
 			)
 		)
-		(property "Footprint" ""
+		(property "Footprint" "smart_compass:JST_S2B-PH-SM4-TB"
 			(at 224.79 41.91 0)
 			(hide yes)
@@
 			)
 		)
-		(property "Footprint" ""
+		(property "Footprint" "smart_compass:SON50P200X200X80-9N"
 			(at 58.42 115.57 0)
 			(hide yes)
@@
 			)
 		)
-		(property "Footprint" ""
+		(property "Footprint" "smart_compass:SOT94P280X100-5N"
 			(at 194.31 58.42 0)
 			(hide yes)
@@
 			)
 		)
-		(property "Footprint" ""
+		(property "Footprint" "smart_compass:SOT95P280X145-5N"
 			(at 71.12 59.69 0)
 			(hide yes)

Commit message: replace capacitor that's in danger of being a bottleneck
Parts:
- C10, C12, C8, C9: DigiKey_PN 1276-6456-1-ND -> 445-6970-1-ND; MPN CL21A106KPFNNNG -> CGA4J3X5R1A106K125AB; Manufacturer Samsung Electro-Mechanics -> TDK; PRICE 0.07 -> 0.24
Changed lines of the file:
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@@
 			)
 		)
-		(property "Datasheet" "https://media.digikey.com/pdf/Data%20Sheets/Samsung%20PDFs/CL_Series_MLCC_ds.pdf"
+		(property "Datasheet" "https://product.tdk.com/system/files/dam/doc/product/capacitor/ceramic/mlcc/catalog/mlcc_automotive_general_en.pdf"
 			(at 236.22 64.77 0)
 			(hide yes)
@@
 			)
 		)
-		(property "MPN" "CL21A106KPFNNNG"
+		(property "MPN" "CGA4J3X5R1A106K125AB"
 			(at 236.22 64.77 90)
 			(hide yes)
@@
 			)
 		)
-		(property "PRICE" "0.07"
+		(property "PRICE" "0.24"
 			(at 236.22 64.77 90)
 			(hide yes)
@@
 			)
 		)
-		(property "Manufacturer" "Samsung Electro-Mechanics"
+		(property "Manufacturer" "TDK"
 			(at 236.22 64.77 0)
 			(hide yes)
@@
 			)
 		)
-		(property "DigiKey_PN" "1276-6456-1-ND"
+		(property "DigiKey_PN" "445-6970-1-ND"
 			(at 236.22 64.77 0)
 			(hide yes)
@@
 			)
 		)
-		(property "Datasheet" "https://media.digikey.com/pdf/Data%20Sheets/Samsung%20PDFs/CL_Series_MLCC_ds.pdf"
+		(property "Datasheet" "https://product.tdk.com/system/files/dam/doc/product/capacitor/ceramic/mlcc/catalog/mlcc_automotive_general_en.pdf"
 			(at 214.63 66.04 0)
 			(hide yes)
@@
 			)
 		)
-		(property "MPN" "CL21A106KPFNNNG"
+		(property "MPN" "CGA4J3X5R1A106K125AB"
 			(at 214.63 66.04 90)
 			(hide yes)
@@
 			)
 		)
-		(property "PRICE" "0.07"
+		(property "PRICE" "0.24"
 			(at 214.63 66.04 90)
 			(hide yes)
@@
 			)
 		)
-		(property "Manufacturer" "Samsung Electro-Mechanics"
+		(property "Manufacturer" "TDK"
 			(at 214.63 66.04 0)
 			(hide yes)
@@
 			)
 		)
-		(property "DigiKey_PN" "1276-6456-1-ND"
+		(property "DigiKey_PN" "445-6970-1-ND"
 			(at 214.63 66.04 0)
 			(hide yes)
@@
 			)
 		)
-		(property "Datasheet" "https://media.digikey.com/pdf/Data%20Sheets/Samsung%20PDFs/CL_Series_MLCC_ds.pdf"
+		(property "Datasheet" "https://product.tdk.com/system/files/dam/doc/product/capacitor/ceramic/mlcc/catalog/mlcc_automotive_general_en.pdf"
 			(at 172.72 66.04 0)
 			(hide yes)
@@
 			)
 		)
-		(property "MPN" "CL21A106KPFNNNG"
+		(property "MPN" "CGA4J3X5R1A106K125AB"
 			(at 172.72 66.04 90)
 			(hide yes)
@@
 			)
 		)
-		(property "PRICE" "0.07"
+		(property "PRICE" "0.24"
 			(at 172.72 66.04 90)
 			(hide yes)
@@
 			)
 		)
-		(property "Manufacturer" "Samsung Electro-Mechanics"
+		(property "Manufacturer" "TDK"
 			(at 172.72 66.04 0)
 			(hide yes)
@@
 			)
 		)
-		(property "DigiKey_PN" "1276-6456-1-ND"
+		(property "DigiKey_PN" "445-6970-1-ND"
 			(at 172.72 66.04 0)
 			(hide yes)
@@
 			)
 		)
-		(property "Datasheet" "https://media.digikey.com/pdf/Data%20Sheets/Samsung%20PDFs/CL_Series_MLCC_ds.pdf"
+		(property "Datasheet" "https://product.tdk.com/system/files/dam/doc/product/capacitor/ceramic/mlcc/catalog/mlcc_automotive_general_en.pdf"
 			(at 236.22 74.93 0)
 			(hide yes)
@@
 			)
 		)
-		(property "MPN" "CL21A106KPFNNNG"
+		(property "MPN" "CGA4J3X5R1A106K125AB"
 			(at 236.22 74.93 90)
 			(hide yes)
@@
 			)
 		)
-		(property "PRICE" "0.07"
+		(property "PRICE" "0.24"
 			(at 236.22 74.93 90)
 			(hide yes)
@@
 			)
 		)
-		(property "Manufacturer" "Samsung Electro-Mechanics"
+		(property "Manufacturer" "TDK"
 			(at 236.22 74.93 0)
 			(hide yes)
@@
 			)
 		)
-		(property "DigiKey_PN" "1276-6456-1-ND"
+		(property "DigiKey_PN" "445-6970-1-ND"
 			(at 236.22 74.93 0)
 			(hide yes)

Commit message: Fixing symbols
Connections:
- net VBUS: now also D1.2 (A); no longer D1.1
- net at C9.1, Q1.2 (S), R9.1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: now also D1.1 (K); no longer D1.2
- no-connect marks 1 -> 0
Changed lines of the file:
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@@
 		(color 0 0 0 0)
 	)
-	(no_connect
-		(at 204.47 60.96)
-	)
 	(wire
 		(pts
@@
 			)
 		)
-		(property "Description" ""
+		(property "Description" "SOT23-5 Fixed Voltage Regulators\n\nPart Current Out V Out V In V Dropout θJA (°C/W) TJ (°C) Digikey Part No.     ADP121   150mA   3.3V   3.4-5.5V   0.09V @ 150mA   --   --   ADP121-AUJZ33R7CT-ND     ADP121   150mA   3.0V   3.1-5.5V   0.09V @ 150mA   --   --   ADP121-AUJZ30R7CT-ND     ADP122   300mA   3.3V   3.4-5.5V   0.085V @ 300mA   --   --   ADP122AUJZ-3.3-R7CT-ND     ADP1712   300mA   3.3V   3.5-5.5V   0.17V @ 300mA   --   --   ADP1712AUJZ-3.3-R7TR-ND     AP7311 (Low Cost)   150mA   3.3V   3.5-6V   0.15V @ 150mA   --   --   AP7311-33WG-7DICT-ND      LD39015M18R   150mA   1.8V   1.9V-5.5V   0.08V @ 100mA   --   --   497-6977-1-ND      LP2985A-33DBVR   150mA   3.3V   3.3-16V   0.28V @ 150mA   206   150   296-18479-1-ND      MCP1824T-3302E/OT   300mA   3.3V   3.5V-6V   0.2V @ 300mA   --   --   MCP1824T-3302E/OTCT-ND      MIC5205-2.5YM5 TR   150mA   2.5V   2.7-16V   0.165V @ 150mA   --   --   576-1257-2-ND     MIC5205-3.0YM5 TR   150mA   3.0V   3.2V-16V   0.165V @ 150mA   --   --   576-1258-2-ND     MIC5205-3.3YM5 TR   150mA   3.3V   3.5V-16V   0.165V @ 150mA   --   --   576-1259-2-ND     TPS780330220   150mA   3.3V+2.2V   3.6-5.5V   250mV Max   --   --   296-23332-1-ND     TDA3663/N1,135   100mA   3.3V   3.5-45V   0.18V @ 50mA   --   --   568-5343-1-ND\n\nMax operating temp can be calculated using θJA, TJ (max junction temperature), and power in watts.  Set the \"Maximum Ambient Temperature\" until it reaches TJ (\"Max Junction Temperature\"), which is the absolute limit for safe use of the regulator: http://www.daycounter.com/Calculators/Heat-Sink-Temperature-Calculator.phtml Heat Sink Temperature Calculator\n\nFor example, With 12V source into a 3.3V LP2985 and a 30mA load, we are dissipating (12V-3.3V) * 0.03A = 0.261W.  With a θJA of 206 °C/W, a TJ of 150°C, and 261mW we can safely use the chip without a heat sink up to 75°C (=147.1°C Junction Temperature)."
 			(at 194.31 58.42 0)
 			(hide yes)

Commit message: Initial placements of main board components. Also set some trace rules
Connections:
- net VSYS: now reaches C9.1, D1.1 (K), Q1.2 (S), R9.1, U3.1 (IN)
Changed lines of the file:
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@@
+		)
+	)
+	(label "VSYS"
+		(at 165.1 55.88 0)
+		(effects
+			(font
+				(size 1.27 1.27)
+			)
+			(justify left bottom)
 		)
 	)
