File: boards/main/user_io.kicad_sch (KiCad schematic)
At the start: 21 parts, among them J3 FH12-10S-0.5SH(55), J4 FH12-10S-0.5SH(55), P1 BUTTON_PADS, U6 BNO086, U7 DRV2605LDGSR

Commit message: exclude non-populated symbols from the BOM
Parts:
- P1, TP1: now left out of the parts list
Changed lines of the file:
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@@
 		(body_style 1)
 		(exclude_from_sim no)
-		(in_bom yes)
+		(in_bom no)
 		(on_board yes)
 		(in_pos_files yes)
@@
 		(body_style 1)
 		(exclude_from_sim no)
-		(in_bom yes)
+		(in_bom no)
 		(on_board yes)
 		(in_pos_files yes)

Commit message: Grab missing footprints and models, and assign them to symbols
Parts:
- U6: footprint (none) -> smart_compass:IC_BNO086
- U7: footprint (none) -> smart_compass:SOP50P490X110-10N
Changed lines of the file:
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@@
 			)
 		)
-		(property "Footprint" ""
+		(property "Footprint" "smart_compass:IC_BNO086"
 			(at 114.3 97.79 0)
 			(hide yes)
@@
 			)
 		)
-		(property "Footprint" ""
+		(property "Footprint" "smart_compass:SOP50P490X110-10N"
 			(at 67.31 156.21 0)
 			(hide yes)

Commit message: replace capacitor that's in danger of being a bottleneck
Parts:
- C19: DigiKey_PN 1276-6456-1-ND -> 445-6970-1-ND; MPN CL21A106KPFNNNG -> CGA4J3X5R1A106K125AB; Manufacturer Samsung Electro-Mechanics -> TDK; PRICE 0.07 -> 0.24
Changed lines of the file:
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@@
 			)
 		)
-		(property "Datasheet" "https://media.digikey.com/pdf/Data%20Sheets/Samsung%20PDFs/CL_Series_MLCC_ds.pdf"
+		(property "Datasheet" "https://product.tdk.com/system/files/dam/doc/product/capacitor/ceramic/mlcc/catalog/mlcc_automotive_general_en.pdf"
 			(at 24.13 148.59 0)
 			(hide yes)
@@
 			)
 		)
-		(property "MPN" "CL21A106KPFNNNG"
+		(property "MPN" "CGA4J3X5R1A106K125AB"
 			(at 24.13 148.59 90)
 			(hide yes)
@@
 			)
 		)
-		(property "PRICE" "0.07"
+		(property "PRICE" "0.24"
 			(at 24.13 148.59 90)
 			(hide yes)
@@
 			)
 		)
-		(property "Manufacturer" "Samsung Electro-Mechanics"
+		(property "Manufacturer" "TDK"
 			(at 24.13 148.59 0)
 			(hide yes)
@@
 			)
 		)
-		(property "DigiKey_PN" "1276-6456-1-ND"
+		(property "DigiKey_PN" "445-6970-1-ND"
 			(at 24.13 148.59 0)
 			(hide yes)

Commit message: Main board PCB layout. No mounting holes yet
Parts:
- added C27, C28: 10pF, Capacitor_SMD:C_0402_1005Metric, symbol smart_compass_main:CAP_CERAMIC0805-NOOUTLINE
- added Y2: 32.768KHZ, smart_compass:XTAL_ABS07-32.768KHZ-7-T, symbol smart_compass_main:ABS07-32.768KHZ-7-T
Connections:
- net GND: now also C27.1, C28.1
- net OSC1: no longer names the net of U6.27 (XIN32)
- net OSC1: now also C27.2, Y2.2
- net OSC2: no longer names the net of U6.26 (XOUT32/CLKSEL1)
- net OSC2: now also C28.2, Y2.1

Commit message: Move the LED ring and haptic engine behind the charge controller, to prevent hot plug ringing from damaging things
Connections:
- net +BATT renamed VSYS
Other:
- moved on the sheet: C14, FB1, R13, TP1
