File: boards/led_ring/LedRing.kicad_sch (KiCad schematic)
At the start: 45 parts, among them J1 FH12-10S-0.5SH(55), U1 TPS61023, U2 74AHCT1G125

Commit message: update the descriptions on the LED ring schematic
Parts:
- D1: Sourcing_Note Run at VDD = 5.0V from the on-board boost U9, which is the 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 -> Run at VDD = 5.0V from the on-board boost converter, which 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
- D16: Sourcing_Note Chain DOUT returns to the main board as NEOPIX_RET. The Inolux typical application circuit recommends a ~500 ohm series resistor at the chain's output terminal as well as its input - R13 covers the input end only. -> Chain DOUT returns to the main board as NEOPIX_RET. The Inolux typical application circuit recommends a ~500 ohm series resistor at the chain's output terminal as well as its input - the main board's 500 ohm series damping resistor covers the input end only.
- J1: Sourcing_Note Vdrive on 1-3, RING_EN on 4, GND on 5, 6, 8, 9, NEOPIX on 7, NEOPIX_RET on 10. Mates with J6 on the main board. Pin 4 was a fourth Vdrive way before the ring moved to a 5V boost; it now carries the enable for U9, which is what lets the MCU disconnect the LEDs' 8mA static draw. Three ways still carry Vdrive, about 370mA at full white, which is well inside a 0.5mm FFC's rating. -> Vdrive on 1-3, RING_EN on 4, GND on 5, 6, 8, 9, NEOPIX on 7, NEOPIX_RET on 10. Mates with the main board's 10-way ring FFC connector. Pin 4 was a fourth Vdrive way before the ring moved to a 5V boost; it now carries the enable for the boost converter, which is what lets the MCU disconnect the LEDs' 8mA static draw. Three ways still carry Vdrive, about 370mA at full white, which is well inside a 0.5mm FFC's rating.
- R1: Sourcing_Note Was a 500R damping resistor when the ring ran at Vdrive. Now the upper leg of a divider: D18's DOUT swings to 5V and must not reach the main board's 3.3V domain. 2.2k/3.9k gives 3.20V at the connector. It still damps the return line at its source end, which is what the 500R was for. -> Was a 500R damping resistor when the ring ran at Vdrive. Now the upper leg of a divider: the last LED in the chain swings its DOUT to 5V, which must not reach the main board's 3.3V domain. 2.2k/3.9k gives 3.20V at the connector. It still damps the return line at its source end, which is what the 500R was for.
- U2: Sourcing_Note Level shifter for NEOPIX. Mandatory at 5V: the Inolux part specifies V_IH = 3.4V minimum at VDD = 5.0V, which 3.3V logic cannot meet. AHCT is the right family because its TTL thresholds (V_IH 2.0V at VCC 5V) accept a 3.3V input directly. OE is tied low so the buffer is always enabled. When RING_EN is low the 5V rail is down and the MCU must hold NEOPIX low too, or it will forward-bias this input's ESD clamp - the main board's R13 (500R) limits that to a few mA, but it is a firmware rule. -> Level shifter for NEOPIX. Mandatory at 5V: the Inolux part specifies V_IH = 3.4V minimum at VDD = 5.0V, which 3.3V logic cannot meet. AHCT is the right family because its TTL thresholds (V_IH 2.0V at VCC 5V) accept a 3.3V input directly. OE is tied low so the buffer is always enabled. When RING_EN is low the 5V rail is down and the MCU must hold NEOPIX low too, or it will forward-bias this input's ESD clamp - the main board's 500R series damping resistor limits that to a few mA, but it is a firmware rule.

Commit message: replace capacitor that's in danger of being a bottleneck
Parts:
- C2: DigiKey_PN 1276-6456-1-ND -> 445-6970-1-ND; MPN CL21A106KPFNNNG -> CGA4J3X5R1A106K125AB; Manufacturer Samsung Electro-Mechanics -> TDK; PRICE (none) -> 0.24
Changed lines of the file:
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@@
 			)
 		)
-    (property "DigiKey_PN" "311-3.90KHRCT-ND" (at 57.15 114.3 0)
-      (effects (font (size 1.27 1.27)) (hide yes))
-    )
+		(property "DigiKey_PN" "311-3.90KHRCT-ND"
+			(at 57.15 114.3 0)
+			(hide yes)
+			(show_name no)
+			(do_not_autoplace no)
+			(effects
+				(font
+					(size 1.27 1.27)
+				)
+			)
+		)
 		(pin "1"
 		)
@@
 			)
 		)
-		(property "Datasheet" "https://media.digikey.com/pdf/Data%20Sheets/Samsung%20PDFs/CL_Series_MLCC_ds.pdf"
+		(property "Datasheet" "https://product.tdk.com/system/files/dam/doc/product/capacitor/ceramic/mlcc/catalog/mlcc_automotive_general_en.pdf"
 			(at 64.77 154.94 0)
 			(hide yes)
@@
 			)
 		)
-		(property "MPN" "CL21A106KPFNNNG"
+		(property "MPN" "CGA4J3X5R1A106K125AB"
 			(at 64.77 154.94 0)
 			(hide yes)
@@
 			)
 		)
-		(property "Manufacturer" "Samsung Electro-Mechanics"
+		(property "Manufacturer" "TDK"
 			(at 64.77 154.94 0)
 			(hide yes)
@@
 			)
 		)
-		(property "DigiKey_PN" "1276-6456-1-ND"
+		(property "DigiKey_PN" "445-6970-1-ND"
 			(at 64.77 154.94 0)
 			(hide yes)
@@
 			)
 		)
+		(property "PRICE" "0.24"
+			(at 64.77 154.94 0)
+			(hide yes)
+			(show_name no)
+			(do_not_autoplace no)
+			(effects
+				(font
+					(size 1.27 1.27)
+				)
+			)
+		)
 		(pin "1"
 		)
@@
 			)
 		)
-    (property "DigiKey_PN" "311-100KHRCT-ND" (at 105.41 191.77 0)
-      (effects (font (size 1.27 1.27)) (hide yes))
-    )
+		(property "DigiKey_PN" "311-100KHRCT-ND"
+			(at 105.41 191.77 0)
+			(hide yes)
+			(show_name no)
+			(do_not_autoplace no)
+			(effects
+				(font
+					(size 1.27 1.27)
+				)
+			)
+		)
 		(pin "1"
 		)

Commit message: start laying out the led ring
Parts:
- renumbered C5 to C1, C1 to C10, C8 to C11, C16 to C13, C20 to C14, C9 to C15, C13 to C16, C21 to C17, C17 to C18, C2 to C19, C10 to C2, C3 to C20, C4 to C21, C14 to C3, C18 to C4, C6 to C5, C15 to C6, C19 to C7, C7 to C8, C11 to C9, D7 to D10, D15 to D12, D4 to D13, D8 to D14, D12 to D15, D5 to D2, D9 to D3, D13 to D4, D2 to D5, D10 to D7, D14 to D8, D3 to D9, U2 to U1, U1 to U2
